File: Aviônica/Aviônica 1.0/esquemático.brd (EAGLE design)
At the start: 160 x 70.8 mm, 9 parts

Commit message: Commit
Parts:
- added U$10, U$11: SWITCH_3PIN, CRD:SWITCH_3PIN
- added U$12, U$8, U$9: JST2.54X2P, CRD:JST2.54X2P_FOOTPRINT
- moved U$4 208.3 mm to (-31.8, 6.35)
- moved U$2 0.76 mm to (134.1, 55.9)
Connections:
- new net BUZZER: U$1.26, U$9.1
- new net ENABLE_SIGNAL: U$1.24, U$10.2
- new net N$4: U$11.1
- new net SKIB1: U$1.28, U$8.1
- new net SKIB2: U$1.27, U$8.2
- new net V_BATTERY: U$11.2, U$12.1
- net GND: now also U$10.1, U$12.2
- net V_3V3: now also U$10.3, U$9.2
- net V_IN: now also U$1.30, U$11.3
Routing:
- added copper zone on layer 16, net GND

Commit message: Push
Parts:
- removed U$4: GPS_ANTENNA, CRD:GPS_ANTENNA_FOOTPRINT
- moved U$5 28.4 mm to (17.4, 42.7)
- moved U$6 25.0 mm to (42.8, 45.2)
- moved U$12 21.6 mm to (110.5, 35.6)
- moved U$10 9.94 mm to (74.0, 40.5)
- moved U$2 7.26 mm to (126.9, 56.4)
- moved U$3 7.24 mm to (127.4, 17.5)
- moved U$11 7.20 mm to (137.7, 35.4)
- moved U$1 3.83 mm to (72.4, 18.2)
- moved U$7 2.34 mm to (33.3, 17.3)
- moved U$9 1.80 mm to (125.7, 35.6)
- moved R1 1.80 mm to (35.6, 16.5)
- moved R2 1.80 mm to (30.5, 16.5)
- moved U$8 1.80 mm to (118.1, 35.6)
Connections:
- net BUZZER: now also U$9.2; no longer U$9.1
- net GND: now also U$8.1
- net SKIB1: now also U$1.29, U$8.2; no longer U$1.28, U$8.1
- net SKIB2: now also U$9.1; no longer U$8.2
- net V_3V3: no longer U$9.2
Other:
- board size 160 x 70.8 mm -> 149.8 x 70.8 mm
