File: Aviônica/Aviônica 1.0/esquemático.sch (EAGLE design)
At the start: 9 parts

Commit message: Commit
Parts:
- added U$10, U$11: SWITCH_3PIN, CRD:SWITCH_3PIN
- added U$12, U$8, U$9: JST2.54X2P, CRD:JST2.54X2P
Connections:
- new net BUZZER: U$1.IO14, U$9.1
- new net ENABLE_SIGNAL: U$1.IO27, U$10.2
- new net N$4: U$11.1
- new net SKIB1: U$1.IO13, U$8.1
- new net SKIB2: U$1.IO12, U$8.2
- new net V_BATTERY: U$11.2, U$12.1
- net GND: now also U$10.1, U$12.2
- net V_3V3: now also U$10.3, U$9.2
- net V_IN: now also U$1.VIN, U$11.3
Other:
- note added: "# Observações: LoRa: Supports 3.3V~5.5V power supply, power supply over 5V can guarantee the best performance."
- note added: "-> Passar por um elevador de tensão 5.0V ->"
- note added: "Alimentação ESP32: A alimentação dessa placa pode ser feita através do próprio conector USB (5,0V) ou então através do pino 5V ou VIN , com uma alimentação regulada de 5,0V. Apesar do Regulador AMS1117 aceitar até 12V na entrada, recomendo que, se for alimentar a placa através desse pino, use sempre uma fonte regulada de 5V, pois assim nunca sobre-aquecerá o mesmo ! Evitando um possível defeito n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"
- moved on the sheet: R1, R2, U$1

Commit message: Push
Parts:
- removed U$4: GPS_ANTENNA, CRD:GPS_ANTENNA
Connections:
- net BUZZER: now also U$9.2; no longer U$9.1
- net GND: now also U$8.1
- net SKIB1: now also U$8.2; no longer U$8.1
- net SKIB2: now also U$9.1; no longer U$8.2
- net V_3V3: no longer U$9.2
Changed lines of the file:
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@@
 <parts>
 <part name="U$1" library="ESP32-DEVKITV1" deviceset="ESP32DEVKITV1" device=""/>
-<part name="U$2" library="CRD" library_urn="urn:adsk.eagle:library:39051337" deviceset="E22-400T30D" device="" package3d_urn="urn:adsk.eagle:package:40965099/2"/>
-<part name="U$3" library="CRD" library_urn="urn:adsk.eagle:library:39051337" deviceset="GPS_MODULE" device="" package3d_urn="urn:adsk.eagle:package:39608400/3"/>
-<part name="U$4" library="CRD" library_urn="urn:adsk.eagle:library:39051337" deviceset="GPS_ANTENNA" device="" package3d_urn="urn:adsk.eagle:package:39608528/1"/>
-<part name="U$5" library="CRD" library_urn="urn:adsk.eagle:library:39051337" deviceset="BMP390" device="V1" package3d_urn="urn:adsk.eagle:package:40965124/3"/>
-<part name="U$6" library="CRD" library_urn="urn:adsk.eagle:library:39051337" deviceset="MPU9250" device="V1" package3d_urn="urn:adsk.eagle:package:40965125/3"/>
+<part name="U$2" library="CRD" library_urn="urn:adsk.eagle:library:39051337" deviceset="E22-400T30D" device="" package3d_urn="urn:adsk.eagle:package:40965099/3"/>
+<part name="U$3" library="CRD" library_urn="urn:adsk.eagle:library:39051337" deviceset="GPS_MODULE" device="" package3d_urn="urn:adsk.eagle:package:39608400/4"/>
+<part name="U$5" library="CRD" library_urn="urn:adsk.eagle:library:39051337" deviceset="BMP390" device="V1" package3d_urn="urn:adsk.eagle:package:40965124/4"/>
+<part name="U$6" library="CRD" library_urn="urn:adsk.eagle:library:39051337" deviceset="MPU9250" device="V1" package3d_urn="urn:adsk.eagle:package:40965125/4"/>
 <part name="U$7" library="CRD" library_urn="urn:adsk.eagle:library:39051337" deviceset="MICROSD_READER" device="" package3d_urn="urn:adsk.eagle:package:39051340/7"/>
 <part name="GND1" library="supply1" library_urn="urn:adsk.eagle:library:371" deviceset="GND" device=""/>
@@
 <instance part="U$2" gate="G$1" x="99.06" y="-20.32" smashed="yes"/>
 <instance part="U$3" gate="G$1" x="-55.88" y="66.04" smashed="yes"/>
-<instance part="U$4" gate="G$1" x="-55.88" y="96.52" smashed="yes"/>
 <instance part="U$5" gate="G$1" x="53.34" y="60.96" smashed="yes"/>
 <instance part="U$6" gate="G$1" x="-2.54" y="63.5" smashed="yes"/>
@@
 <wire x1="172.83905625" y1="20.071934375" x2="175.26" y2="20.071934375" width="0.1524" layer="91"/>
 </segment>
+<segment>
+<pinref part="U$8" gate="G$1" pin="1"/>
+<wire x1="167.64" y1="-22.86" x2="167.64" y2="-25.4" width="0.1524" layer="91"/>
+<label x="167.64" y="-33.02" size="1.778" layer="95" rot="R90"/>
+</segment>
 </net>
 <net name="V_IN" class="0">
@@
 </segment>
 <segment>
-<pinref part="U$9" gate="G$1" pin="2"/>
-<wire x1="193.04" y1="-22.86" x2="193.04" y2="-25.4" width="0.1524" layer="91"/>
-<label x="193.04" y="-30.48" size="1.778" layer="95" rot="R90"/>
-</segment>
-<segment>
 <pinref part="U$10" gate="G$1" pin="3"/>
 <wire x1="185.42" y1="27.94" x2="185.42" y2="20.32" width="0.1524" layer="91"/>
@@
 <net name="SKIB1" class="0">
 <segment>
-<pinref part="U$8" gate="G$1" pin="1"/>
-<wire x1="167.64" y1="-22.86" x2="167.64" y2="-25.4" width="0.1524" layer="91"/>
-<label x="167.64" y="-33.02" size="1.778" layer="95" rot="R90"/>
-</segment>
-<segment>
 <pinref part="U$1" gate="G$1" pin="IO13"/>
 <wire x1="-48.26" y1="-58.42" x2="-53.34" y2="-58.42" width="0.1524" layer="91"/>
 <label x="-58.42" y="-58.42" size="1.778" layer="95"/>
 </segment>
-</net>
-<net name="SKIB2" class="0">
 <segment>
 <pinref part="U$8" gate="G$1" pin="2"/>
@@
 <label x="172.72" y="-33.02" size="1.778" layer="95" rot="R90"/>
 </segment>
+</net>
+<net name="SKIB2" class="0">
 <segment>
 <pinref part="U$1" gate="G$1" pin="IO12"/>
@@
 <label x="-58.42" y="-55.88" size="1.778" layer="95"/>
 </segment>
-</net>
-<net name="BUZZER" class="0">
 <segment>
 <pinref part="U$9" gate="G$1" pin="1"/>
@@
 <label x="187.96" y="-33.02" size="1.778" layer="95" rot="R90"/>
 </segment>
+</net>
+<net name="BUZZER" class="0">
 <segment>
 <pinref part="U$1" gate="G$1" pin="IO14"/>
@@
 <label x="-58.42" y="-53.34" size="1.778" layer="95"/>
 </segment>
-</net>
+<segment>
+<pinref part="U$9" gate="G$1" pin="2"/>
+<wire x1="193.04" y1="-22.86" x2="193.04" y2="-25.4" width="0.1524" layer="91"/>
+<label x="193.04" y="-33.02" size="1.778" layer="95" rot="R90"/>
+</segment>
+</net>
