File: Aviônica/Aviônica 2.0/esquemático.brd (EAGLE design)
At the start: 149.8 x 70.8 mm, 13 parts

Commit message: Message
Parts:
- removed R1, R2: 330, rcl:0207/10
- removed U$10: SWITCH_3PIN, CRD:SWITCH_3PIN
- added U$5: SWITCH_ALAVANCA, CRD:SWITCH_ALAVANCA_FOOTPRINT
- moved U$12 18.2 mm to (128.7, 35.6)
- moved U$9 15.2 mm to (110.5, 35.6)
- moved U$11 2.54 mm to (140.2, 35.4)
- moved U$3 1.93 mm to (129.2, 16.8), flipped to the bottom, turned to 90 degrees
- moved U$2 1.27 mm to (126.9, 56.4)
- moved U$8 0.76 mm to (118.9, 35.6)
Connections:
- net TX3_ESP renamed TX1_ESP
- removed net N$1: R1.2, U$7.MOSI
- removed net N$2: R2.2, U$7.MISO
- removed net N$3: U$2.AUX
- removed net N$4: U$11.1
- removed net RX3_ESP: U$1.4, U$3.TX
- new net M0: U$1.20, U$2.M0
- new net M1: U$1.19, U$2.M1
- new net RX1_ESP: U$1.3, U$3.TX
- net ENABLE_SIGNAL: now also U$5.PIN2; no longer U$10.2
- net GND: now also U$5.PIN1; no longer U$10.1, U$2.M0, U$2.M1
- net MISO: now also U$7.MISO; no longer R2.1
- net MOSI: now also U$7.MOSI; no longer R1.1
- net V_3V3: now also U$5.PIN3, U$7.VCC; no longer U$10.3
Routing:
- net V_3V3: track 0.00 -> 159.3 mm, vias 0 -> 3
- net SDA: track 0.00 -> 116.5 mm
- net M1: track 0.00 -> 110.0 mm
- net M0: track 0.00 -> 105.5 mm
- net V_IN: track 0.00 -> 103.0 mm
- net ENABLE_SIGNAL: track 0.00 -> 102.7 mm, vias 0 -> 1
- net BUZZER: track 0.00 -> 76.2 mm
- net RX2_ESP: track 0.00 -> 74.1 mm
- net TX2_ESP: track 0.00 -> 73.5 mm, vias 0 -> 1
- net SKIB1: track 0.00 -> 72.2 mm
- net SKIB2: track 0.00 -> 66.5 mm
- net SCL: track 0.00 -> 63.3 mm, vias 0 -> 1
- net TX1_ESP: track 0.00 -> 57.2 mm
- net SCK: track 0.00 -> 55.3 mm
- net CS: track 0.00 -> 54.9 mm, vias 0 -> 2
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- added copper zone on layer 16, net ANTENNA
