File: Aviônica/Aviônica 2.0/esquemático.sch (EAGLE design)
At the start: 13 parts

Commit message: Message
Parts:
- removed R1, R2: 330, rcl:R-EU_0207/10
- removed U$10: SWITCH_3PIN, CRD:SWITCH_3PIN
- added U$5: SWITCH_ALAVANCA, CRD:SWITCH_ALAVANCA
Connections:
- net TX3_ESP renamed TX1_ESP
- removed net N$1: R1.2, U$7.MOSI
- removed net N$2: R2.2, U$7.MISO
- removed net N$3: U$2.AUX
- removed net N$4: U$11.1
- removed net RX3_ESP: U$1.IO2, U$3.TX
- new net M0: U$1.IO35, U$2.M0
- new net M1: U$1.IO34, U$2.M1
- new net RX1_ESP: U$1.IO15, U$3.TX
- net ENABLE_SIGNAL: now also U$5.PIN2; no longer U$10.2
- net GND: now also U$5.PIN1; no longer U$10.1, U$2.M0, U$2.M1
- net MISO: now also U$7.MISO; no longer R2.1
- net MOSI: now also U$7.MOSI; no longer R1.1
- net V_3V3: now also U$5.PIN3, U$7.VCC; no longer U$10.3
