File: Paraquedas/Paraquedas 1.1/Esquema.brd (EAGLE design)
At the start: 51.5 x 57 mm, 9 parts, among them Q1 IRF540, Q2 IRF540, Q3 IRF540

Commit message: Message
Connections:
- new net 3V3: U$1.2
- net BUZZER: now also U$1.1; no longer U$2.2
- net GND: no longer U$1.1
- net SKIB1: now also U$2.1; no longer U$1.2
- net SKIB2: now also U$2.2; no longer U$2.1
Routing:
- net BUZZER: track 44.8 -> 34.0 mm
- net SKIB1: track 17.2 -> 22.7 mm
- net SKIB2: track 11.4 -> 12.4 mm
Changed lines of the file:
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@@
 </layers>
 <board>
-<fusionsync huburn="a.YnVzaW5lc3M6ZGlzY2VudGU3MA" projecturn="a.YnVzaW5lc3M6ZGlzY2VudGU3MCMyMDIyMDIxNzQ5ODU5MDQ4MQ" f3durn="urn:adsk.wipprod:dm.lineage:eC2E5IMDRm2aw-eJDvErbw" pcbguid="" lastpulledtime="" lastsyncedchangeguid="" latestrevisionid="d5523bd2-7437-4db2-b767-71d2d1ac56fe" lastsyncedrevisionid="d5523bd2-7437-4db2-b767-71d2d1ac56fe" lastboardhashguid="33d128af-a64a-b0db-033b-a1b71b82984a" lastpushedtime="2023-05-09T12:36:54Z" linktopcb3d="false"/>
+<fusionsync huburn="a.YnVzaW5lc3M6ZGlzY2VudGU3MA" projecturn="a.YnVzaW5lc3M6ZGlzY2VudGU3MCMyMDIyMDIxNzQ5ODU5MDQ4MQ" f3durn="urn:adsk.wipprod:dm.lineage:eC2E5IMDRm2aw-eJDvErbw" pcbguid="" lastpulledtime="" lastsyncedchangeguid="" latestrevisionid="d5523bd2-7437-4db2-b767-71d2d1ac56fe" lastsyncedrevisionid="d5523bd2-7437-4db2-b767-71d2d1ac56fe" lastboardhashguid="33d128af-a64a-b0db-033b-a1b71b82984a" lastpushedtime="2023-05-09T12:36:54Z" linktopcb3d="true"/>
 <plain>
 <wire x1="50.5" y1="-3" x2="-1" y2="-3" width="0" layer="20"/>
@@
 <signal name="BUZZER">
 <contactref element="Q3" pad="1"/>
-<wire x1="23.5" y1="-0.5" x2="39.4" y2="-0.5" width="1" layer="16"/>
 <wire x1="21" y1="2" x2="21" y2="8" width="1" layer="16"/>
 <wire x1="21" y1="8" x2="17.0264" y2="11.9736" width="1" layer="16"/>
@@
 <wire x1="13" y1="12" x2="11.46" y2="13.54" width="1" layer="16"/>
 <wire x1="11.46" y1="13.54" x2="11.46" y2="14.65" width="1" layer="16"/>
-<wire x1="23.5" y1="-0.5" x2="21" y2="2" width="1" layer="16"/>
-<contactref element="U$2" pad="2"/>
-<wire x1="42.77" y1="2.87" x2="42.77" y2="4.5" width="1" layer="16"/>
-<wire x1="39.4" y1="-0.5" x2="42.77" y2="2.87" width="1" layer="16"/>
+<wire x1="21" y1="2" x2="23.5" y2="-0.5" width="1" layer="16"/>
+<contactref element="U$1" pad="1"/>
+<wire x1="23.5" y1="-0.5" x2="29.1" y2="-0.5" width="1" layer="16"/>
+<wire x1="29.1" y1="-0.5" x2="31.2" y2="1.6" width="1" layer="16"/>
+<wire x1="31.2" y1="1.6" x2="31.2" y2="4.43" width="1" layer="16"/>
+<wire x1="31.2" y1="4.43" x2="31.13" y2="4.5" width="1" layer="16"/>
 </signal>
 <signal name="GND">
@@
 <vertex x="0" y="53"/>
 </polygon>
-<contactref element="U$1" pad="1"/>
 </signal>
 <signal name="SKIB1">
@@
 <wire x1="24" y1="11" x2="24" y2="14.65" width="1" layer="16"/>
 <wire x1="24" y1="14.65" x2="24.07" y2="14.72" width="1" layer="16"/>
-<wire x1="30" y1="10" x2="32.17" y2="7.83" width="1.016" layer="16"/>
-<wire x1="32.17" y1="7.83" x2="33.7" y2="6.3" width="1" layer="16"/>
-<contactref element="U$1" pad="2"/>
-<wire x1="33.7" y1="6.3" x2="33.7" y2="4.53" width="1" layer="16"/>
-<wire x1="33.7" y1="4.53" x2="33.67" y2="4.5" width="1" layer="16"/>
+<contactref element="U$2" pad="1"/>
+<wire x1="30" y1="10" x2="34.2" y2="10" width="1" layer="16"/>
+<wire x1="39.7" y1="4.5" x2="40.23" y2="4.5" width="1" layer="16"/>
+<wire x1="34.2" y1="10" x2="39.7" y2="4.5" width="1" layer="16"/>
 </signal>
 <signal name="VCC">
@@
 <contactref element="Q2" pad="1"/>
 <wire x1="37.47" y1="14.72" x2="37.47" y2="10.53" width="1" layer="16"/>
-<wire x1="37.47" y1="10.53" x2="40.2" y2="7.8" width="1" layer="16"/>
-<contactref element="U$2" pad="1"/>
-<wire x1="40.2" y1="4.53" x2="40.23" y2="4.5" width="1" layer="16"/>
-<wire x1="40.2" y1="7.8" x2="40.2" y2="4.53" width="1" layer="16"/>
+<contactref element="U$2" pad="2"/>
+<wire x1="42.77" y1="5.23" x2="42.77" y2="4.5" width="1" layer="16"/>
+<wire x1="37.47" y1="10.53" x2="42.77" y2="5.23" width="1" layer="16"/>
 </signal>
 <signal name="N$2">
@@
 </polygon>
 </signal>
+<signal name="3V3">
+<contactref element="U$1" pad="2"/>
+</signal>
 </signals>
