File: Paraquedas/Paraquedas 1.1/Esquema.sch (EAGLE design)
At the start: 9 parts, among them Q1 IRF540, Q2 IRF540, Q3 IRF540

Commit message: Message
Connections:
- new net 3V3: U$1.2
- net BUZZER: now also U$1.1; no longer U$2.2
- net GND: no longer U$1.1
- net SKIB1: now also U$2.1; no longer U$1.2
- net SKIB2: now also U$2.2; no longer U$2.1
Changed lines of the file:
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@@
 </segment>
 <segment>
-<pinref part="U$2" gate="G$1" pin="2"/>
-<wire x1="27.94" y1="-2.54" x2="27.94" y2="-12.7" width="0.1524" layer="91"/>
-<label x="27.94" y="-12.7" size="1.778" layer="95" rot="R90"/>
+<pinref part="U$1" gate="G$1" pin="1"/>
+<wire x1="22.86" y1="38.1" x2="22.86" y2="27.94" width="0.1524" layer="91"/>
+<label x="22.86" y="22.86" size="1.778" layer="95" rot="R90"/>
 </segment>
 </net>
@@
 <wire x1="68.58" y1="7.62" x2="68.58" y2="15.24" width="0.1524" layer="91"/>
 </segment>
-<segment>
-<pinref part="U$1" gate="G$1" pin="1"/>
-<wire x1="22.86" y1="38.1" x2="22.86" y2="27.94" width="0.1524" layer="91"/>
-<label x="22.86" y="22.86" size="1.778" layer="95" rot="R90"/>
-</segment>
 </net>
 <net name="SKIB1" class="0">
@@
 </segment>
 <segment>
-<pinref part="U$1" gate="G$1" pin="2"/>
-<wire x1="27.94" y1="38.1" x2="27.94" y2="27.94" width="0.1524" layer="91"/>
-<label x="27.94" y="22.86" size="1.778" layer="95" rot="R90"/>
+<pinref part="U$2" gate="G$1" pin="1"/>
+<wire x1="22.86" y1="-2.54" x2="22.86" y2="-12.7" width="0.1524" layer="91"/>
+<label x="22.86" y="-12.7" size="1.778" layer="95" rot="R90"/>
 </segment>
 </net>
@@
 </segment>
 <segment>
-<pinref part="U$2" gate="G$1" pin="1"/>
-<wire x1="22.86" y1="-2.54" x2="22.86" y2="-12.7" width="0.1524" layer="91"/>
-<label x="22.86" y="-12.7" size="1.778" layer="95" rot="R90"/>
+<pinref part="U$2" gate="G$1" pin="2"/>
+<wire x1="27.94" y1="-2.54" x2="27.94" y2="-12.7" width="0.1524" layer="91"/>
+<label x="27.94" y="-12.7" size="1.778" layer="95" rot="R90"/>
 </segment>
 </net>
@@
 </segment>
 </net>
+<net name="3V3" class="0">
+<segment>
+<pinref part="U$1" gate="G$1" pin="2"/>
+<wire x1="27.94" y1="38.1" x2="27.94" y2="27.94" width="0.1524" layer="91"/>
+<label x="27.94" y="22.86" size="1.778" layer="95" rot="R90"/>
+</segment>
+</net>
