File: Aviônica/Avionica 2.2/Avionicapart1.brd (EAGLE design)
At the start: 100 x 70.8 mm, 12 parts, among them J1 MICRO-SD-PUSH-PUSH-EXT-PIN, U1 ESP32-DEVKIT-V1

Commit message: Atualização-avionica
Parts:
- removed 3.3-BUZ: (no value), SparkFun-Connectors:1X02_2.54_SCREWTERM
- removed U$5: SWITCH_ALAVANCA, CRD:SWITCH_ALAVANCA_FOOTPRINT
- added 3.3-BUZ1, EN-3.3V: (no value), SparkFun-Connectors:1X02_2.54_SCREWTERM
- moved GPS-G-V 2.25 mm to (128.7, 46.5)
- moved GPS-TX-RX 0.61 mm to (128.9, 33.6), turned to 270 degrees
Connections:
- net BUZZER: now also EN-3.3V.P2; no longer 3.3-BUZ.P2
- net ENABLE_SIGNAL: now also 3.3-BUZ1.P1; no longer U$5.PIN2
- net GND: no longer U$5.PIN1
- net RX1_ESP: now also GPS-TX-RX.P2; no longer GPS-TX-RX.P1
- net TX1_ESP: now also GPS-TX-RX.P1; no longer GPS-TX-RX.P2
- net V_3V3: now also 3.3-BUZ1.P2, EN-3.3V.P1; no longer 3.3-BUZ.P1, U$5.PIN3
Routing:
- net V_3V3: track 94.5 -> 103.2 mm
- net ENABLE_SIGNAL: track 60.5 -> 66.9 mm, vias 1 -> 0
- net BUZZER: track 61.9 -> 63.2 mm
- net TX1_ESP: track 54.8 -> 53.7 mm
- net RX1_ESP: track 51.5 -> 50.5 mm
