File: Aviônica/Avionica 2.2/Avionicapart1.brd (EAGLE design)
At the start: 100 x 70.8 mm, 12 parts, among them J1 MICRO-SD-PUSH-PUSH-EXT-PIN, U1 ESP32-DEVKIT-V1

Commit message: correções avionica e paraquedas
Parts:
- added GND, SK1-SK2: (no value), SparkFun-Connectors:1X02_2.54_SCREWTERM
Connections:
- new net SK1: SK1-SK2.P1, U1.23
- new net SK2: SK1-SK2.P2, U1.24
- net GND: now also GND.P1, GND.P2
Routing:
- net SK1: track 0.00 -> 62.7 mm
- net SK2: track 0.00 -> 58.2 mm
- net ENABLE_SIGNAL: track 66.9 -> 64.9 mm

Commit message: update
Parts:
- removed 3.3-BUZ1: (no value), SparkFun-Connectors:1X02_2.54_SCREWTERM
- added 3.3V-BUZ: (no value), SparkFun-Connectors:1X02_2.54_SCREWTERM
- moved EN-3.3V 12.8 mm to (128.8, 40.2)
- moved SKIB2-SKIB1 1.36 mm to (137.8, 52.9)
- moved GND 0.86 mm to (135.9, 31.9)
Connections:
- net BUZZER: now also 3.3V-BUZ.P2; no longer EN-3.3V.P2
- net ENABLE_SIGNAL: now also EN-3.3V.P1; no longer 3.3-BUZ1.P1
- net V_3V3: now also 3.3V-BUZ.P1, EN-3.3V.P2; no longer 3.3-BUZ1.P2, EN-3.3V.P1
Routing:
- net SKIB2: track 46.9 -> 45.5 mm
- net SKIB1: track 41.9 -> 40.5 mm
Changed lines of the file:
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@@
 <rectangle x1="169.788028125" y1="76.40985625" x2="169.805809375" y2="76.4182375" layer="22" rot="R180"/>
 <rectangle x1="169.795646875" y1="76.4182375" x2="169.805809375" y2="76.426875" layer="22" rot="R180"/>
+<hole x="149.0504" y="24.833275" drill="1"/>
 </plain>
 <attributes>
@@
 <attribute name="VALUE" x="124.60763125" y="47.811421875" size="0.6096" layer="27" font="vector" ratio="20" rot="R270"/>
 </element>
-<element name="EN-3.3V" library="SparkFun-Connectors" package="1X02_2.54_SCREWTERM" value="" x="128.62580625" y="52.966696875" smashed="yes" rot="R270">
-<attribute name="NAME" x="124.2408875" y="54.056609375" size="0.8128" layer="25" font="vector" ratio="20" rot="R270"/>
+<element name="3.3V-BUZ" library="SparkFun-Connectors" package="1X02_2.54_SCREWTERM" value="" x="128.62580625" y="52.966696875" smashed="yes" rot="R270">
+<attribute name="NAME" x="132.436884375" y="54.361103125" size="0.8128" layer="25" font="vector" ratio="20" rot="R270"/>
 <attribute name="VALUE" x="124.56180625" y="54.236696875" size="0.6096" layer="27" font="vector" ratio="20" rot="R270"/>
 </element>
-<element name="SKIB2-SKIB1" library="SparkFun-Connectors" package="1X02_2.54_SCREWTERM" value="" x="136.5" y="52.4" smashed="yes" rot="R270">
-<attribute name="NAME" x="140.029" y="54.47" size="0.8128" layer="25" font="vector" ratio="20" rot="R270"/>
-<attribute name="VALUE" x="132.436" y="53.67" size="0.6096" layer="27" font="vector" ratio="20" rot="R270"/>
+<element name="SKIB2-SKIB1" library="SparkFun-Connectors" package="1X02_2.54_SCREWTERM" value="" x="137.785646875" y="52.85674375" smashed="yes" rot="R270">
+<attribute name="NAME" x="141.314646875" y="54.92674375" size="0.8128" layer="25" font="vector" ratio="20" rot="R270"/>
+<attribute name="VALUE" x="133.721646875" y="54.12674375" size="0.6096" layer="27" font="vector" ratio="20" rot="R270"/>
 </element>
 <element name="GND-BAT" library="SparkFun-Connectors" package="1X02_2.54_SCREWTERM" value="" x="216.1" y="40.3" smashed="yes" rot="R90">
@@
 <attribute name="VALUE" x="220.164" y="39.03" size="0.6096" layer="27" font="vector" ratio="20" rot="R90"/>
 </element>
-<element name="3.3-BUZ1" library="SparkFun-Connectors" package="1X02_2.54_SCREWTERM" value="" x="128.75918125" y="40.151075" smashed="yes" rot="R270">
+<element name="EN-3.3V" library="SparkFun-Connectors" package="1X02_2.54_SCREWTERM" value="" x="128.75918125" y="40.151075" smashed="yes" rot="R270">
 <attribute name="NAME" x="132.441925" y="41.65790625" size="0.8128" layer="25" font="vector" ratio="20" rot="R270"/>
 <attribute name="VALUE" x="124.69518125" y="41.421075" size="0.6096" layer="27" font="vector" ratio="20" rot="R270"/>
 </element>
-<element name="GND" library="SparkFun-Connectors" package="1X02_2.54_SCREWTERM" value="" x="136.642221875" y="32.42028125" smashed="yes">
-<attribute name="NAME" x="136.674784375" y="28.00853125" size="0.8128" layer="25" font="vector" ratio="20"/>
-<attribute name="VALUE" x="135.372221875" y="28.35628125" size="0.6096" layer="27" font="vector" ratio="20"/>
+<element name="GND" library="SparkFun-Connectors" package="1X02_2.54_SCREWTERM" value="" x="135.940190625" y="31.92124375" smashed="yes">
+<attribute name="NAME" x="135.972753125" y="27.50949375" size="0.8128" layer="25" font="vector" ratio="20"/>
+<attribute name="VALUE" x="134.670190625" y="27.85724375" size="0.6096" layer="27" font="vector" ratio="20"/>
 </element>
 <element name="SK1-SK2" library="SparkFun-Connectors" package="1X02_2.54_SCREWTERM" value="" x="137.369625" y="40.345615625" smashed="yes" rot="R270">
@@
 <wire x1="128.67163125" y1="46.541421875" x2="128.813053125" y2="46.4" width="1.8" layer="16"/>
 <wire x1="131" y1="46.4" x2="128.813053125" y2="46.4" width="1.8" layer="16"/>
-<contactref element="EN-3.3V" pad="P1"/>
+<contactref element="3.3V-BUZ" pad="P1"/>
 <wire x1="128.62580625" y1="50.426696875" x2="128.62580625" y2="48.77419375" width="1.8" layer="16"/>
 <wire x1="128.62580625" y1="48.77419375" x2="131" y2="46.4" width="1.8" layer="16"/>
-<contactref element="3.3-BUZ1" pad="P2"/>
+<contactref element="EN-3.3V" pad="P2"/>
 <wire x1="128.75918125" y1="40.151075" x2="133.590496875" y2="40.151075" width="1.27" layer="16"/>
 <wire x1="133.590496875" y1="40.151075" x2="139.839421875" y2="46.4" width="1.27" layer="16"/>
@@
 <wire x1="175" y1="56.8" x2="175" y2="58.365" width="0.6096" layer="1"/>
 <wire x1="175" y1="58.365" x2="174.965" y2="58.4" width="0.6096" layer="1"/>
-<wire x1="173.206528125" y1="55.006528125" x2="139.106528125" y2="55.006528125" width="0.6096" layer="1"/>
+<wire x1="173.206528125" y1="55.006528125" x2="140.552878125" y2="55.006528125" width="0.6096" layer="1"/>
 <contactref element="SKIB2-SKIB1" pad="P2"/>
-<wire x1="139.106528125" y1="55.006528125" x2="136.5" y2="52.4" width="0.6096" layer="1"/>
+<wire x1="140.552878125" y1="55.006528125" x2="138.40309375" y2="52.85674375" width="0.6096" layer="1"/>
+<wire x1="138.40309375" y1="52.85674375" x2="137.785646875" y2="52.85674375" width="0.6096" layer="1"/>
 </signal>
 <signal name="SKIB2">
 <contactref element="U1" pad="27"/>
-<wire x1="176.705559375" y1="53.505559375" x2="140.905559375" y2="53.505559375" width="0.6096" layer="1"/>
+<wire x1="176.705559375" y1="53.505559375" x2="142.005121875" y2="53.505559375" width="0.6096" layer="1"/>
 <wire x1="176.705559375" y1="53.505559375" x2="177.505" y2="54.305" width="0.6096" layer="1"/>
 <wire x1="177.505" y1="54.305" x2="177.505" y2="58.4" width="0.6096" layer="1"/>
 <contactref element="SKIB2-SKIB1" pad="P1"/>
-<wire x1="140.905559375" y1="53.505559375" x2="137.26" y2="49.86" width="0.6096" layer="1"/>
-<wire x1="137.26" y1="49.86" x2="136.5" y2="49.86" width="0.6096" layer="1"/>
+<wire x1="142.005121875" y1="53.505559375" x2="138.81630625" y2="50.31674375" width="0.6096" layer="1"/>
+<wire x1="137.785646875" y1="50.31674375" x2="138.81630625" y2="50.31674375" width="0.6096" layer="1"/>
 </signal>
 <signal name="BUZZER">
@@
 <wire x1="133.4" y1="46.4" x2="137.1" y2="46.4" width="0.6096" layer="1"/>
 <wire x1="137.1" y1="46.4" x2="142.64785" y2="51.94785" width="0.6096" layer="1"/>
-<contactref element="EN-3.3V" pad="P2"/>
+<contactref element="3.3V-BUZ" pad="P2"/>
 <wire x1="131.8" y1="50.6" x2="129.433303125" y2="52.966696875" width="0.6096" layer="1"/>
 <wire x1="129.433303125" y1="52.966696875" x2="128.62580625" y2="52.966696875" width="0.6096" layer="1"/>
@@
 <wire x1="143.3279375" y1="50.5279375" x2="140.4" y2="47.6" width="0.6096" layer="1"/>
 <wire x1="140.4" y1="47.6" x2="140.4" y2="47.4678625" width="0.6096" layer="1"/>
-<contactref element="3.3-BUZ1" pad="P1"/>
+<contactref element="EN-3.3V" pad="P1"/>
 <wire x1="140.4" y1="47.4678625" x2="130.596503125" y2="37.664365625" width="0.6096" layer="1"/>
 <wire x1="128.812471875" y1="37.664365625" x2="128.75918125" y2="37.611075" width="0.6096" layer="1"/>
