File: Aviônica/Avionica 2.2/Avionicapart1.sch (EAGLE design)
At the start: 12 parts, among them J1 MICRO-SD-PUSH-PUSH-EXT-PIN, U1 ESP32-DEVKIT-V1

Commit message: Atualização-avionica
Parts:
- removed U$5: SWITCH_ALAVANCA, CRD:SWITCH_ALAVANCA
- added 3.3-BUZ1: (no value), SparkFun-Connectors:CONN_022.54MM_SCREWTERM
- renumbered 3.3-BUZ to EN-3.3V
Connections:
- net ENABLE_SIGNAL: now also 3.3-BUZ1.1; no longer U$5.PIN2
- net GND: no longer U$5.PIN1
- net RX1_ESP: now also GPS-TX-RX.2; no longer GPS-TX-RX.1
- net TX1_ESP: now also GPS-TX-RX.1; no longer GPS-TX-RX.2
- net V_3V3: now also 3.3-BUZ1.2; no longer U$5.PIN3
Changed lines of the file:
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@@
 <part name="U$4" library="CRD" library_urn="urn:adsk.eagle:library:39051337" deviceset="BMP280" device="V1" package3d_urn="urn:adsk.eagle:package:39029072/5"/>
 <part name="U$6" library="CRD" library_urn="urn:adsk.eagle:library:39051337" deviceset="MPU6050" device="V1" package3d_urn="urn:adsk.eagle:package:39029071/7"/>
-<part name="U$5" library="CRD" library_urn="urn:adsk.eagle:library:39051337" deviceset="SWITCH_ALAVANCA" device=""/>
-<part name="GND10" library="supply1" library_urn="urn:adsk.eagle:library:371" deviceset="GND" device=""/>
 <part name="U1" library="ESP32-DEVKIT-V1" deviceset="ESP32-DEVKIT-V1" device=""/>
 <part name="GND8" library="supply1" library_urn="urn:adsk.eagle:library:371" deviceset="GND" device=""/>
@@
 <part name="GPS-TX-RX" library="SparkFun-Connectors" deviceset="CONN_02" device="2.54MM_SCREWTERM"/>
 <part name="GPS-G-V" library="SparkFun-Connectors" deviceset="CONN_02" device="2.54MM_SCREWTERM"/>
-<part name="3.3-BUZ" library="SparkFun-Connectors" deviceset="CONN_02" device="2.54MM_SCREWTERM"/>
+<part name="EN-3.3V" library="SparkFun-Connectors" deviceset="CONN_02" device="2.54MM_SCREWTERM"/>
 <part name="SKIB2-SKIB1" library="SparkFun-Connectors" deviceset="CONN_02" device="2.54MM_SCREWTERM"/>
 <part name="GND-BAT" library="SparkFun-Connectors" deviceset="CONN_02" device="2.54MM_SCREWTERM"/>
+<part name="3.3-BUZ1" library="SparkFun-Connectors" deviceset="CONN_02" device="2.54MM_SCREWTERM"/>
 </parts>
 <sheets>
@@
 <instance part="U$4" gate="G$1" x="48.26" y="68.58" smashed="yes"/>
 <instance part="U$6" gate="G$1" x="-7.62" y="66.04" smashed="yes"/>
-<instance part="U$5" gate="G$1" x="180.34" y="40.64" smashed="yes"/>
-<instance part="GND10" gate="1" x="175.37905625" y="14.991934375" smashed="yes">
-<attribute name="VALUE" x="172.83905625" y="12.451934375" size="1.778" layer="96"/>
-</instance>
 <instance part="U1" gate="G$1" x="-25.4" y="-53.34" smashed="yes">
 <attribute name="VALUE" x="-35.56" y="-83.82" size="1.778" layer="96"/>
@@
 <attribute name="NAME" x="-55.372" y="99.06" size="1.778" layer="95" font="vector" rot="R270"/>
 </instance>
-<instance part="3.3-BUZ" gate="G$1" x="167.64" y="-10.16" smashed="yes" rot="R270">
+<instance part="EN-3.3V" gate="G$1" x="167.64" y="-10.16" smashed="yes" rot="R270">
 <attribute name="VALUE" x="162.814" y="-7.62" size="1.778" layer="96" font="vector" rot="R270"/>
 <attribute name="NAME" x="173.228" y="-7.62" size="1.778" layer="95" font="vector" rot="R270"/>
@@
 <attribute name="VALUE" x="162.814" y="96.52" size="1.778" layer="96" font="vector" rot="R270"/>
 <attribute name="NAME" x="173.228" y="96.52" size="1.778" layer="95" font="vector" rot="R270"/>
+</instance>
+<instance part="3.3-BUZ1" gate="G$1" x="185.42" y="2.54" smashed="yes" rot="R90">
+<attribute name="VALUE" x="190.246" y="0" size="1.778" layer="96" font="vector" rot="R90"/>
+<attribute name="NAME" x="179.832" y="0" size="1.778" layer="95" font="vector" rot="R90"/>
 </instance>
 </instances>
@@
 </segment>
 <segment>
-<pinref part="U$5" gate="G$1" pin="PIN1"/>
-<pinref part="GND10" gate="1" pin="GND"/>
-<wire x1="175.26" y1="30.48" x2="175.37905625" y2="27.94" width="0.1524" layer="91"/>
-<wire x1="175.37905625" y1="27.94" x2="175.37905625" y2="17.531934375" width="0.1524" layer="91"/>
-</segment>
-<segment>
 <pinref part="U1" gate="G$1" pin="GND"/>
 <pinref part="GND8" gate="1" pin="GND"/>
@@
 </segment>
 <segment>
-<pinref part="U$5" gate="G$1" pin="PIN3"/>
-<wire x1="185.42" y1="30.48" x2="185.42" y2="15.24" width="0.1524" layer="91"/>
-<label x="185.42" y="12.7" size="1.778" layer="95" rot="R90"/>
-</segment>
-<segment>
 <pinref part="U1" gate="G$1" pin="3V3"/>
 <wire x1="-10.16" y1="-27.94" x2="-2.54" y2="-27.94" width="0.1524" layer="91"/>
@@
 </segment>
 <segment>
-<pinref part="3.3-BUZ" gate="G$1" pin="1"/>
+<pinref part="EN-3.3V" gate="G$1" pin="1"/>
 <wire x1="167.64" y1="-17.78" x2="167.64" y2="-22.86" width="0.1524" layer="91"/>
 <label x="167.64" y="-22.86" size="1.4224" layer="95" rot="R270" xref="yes"/>
+</segment>
+<segment>
+<pinref part="3.3-BUZ1" gate="G$1" pin="2"/>
+<wire x1="182.88" y1="10.16" x2="182.88" y2="15.24" width="0.1524" layer="91"/>
+<label x="180.34" y="12.7" size="1.778" layer="95" rot="R90"/>
 </segment>
 </net>
@@
 </segment>
 <segment>
-<pinref part="3.3-BUZ" gate="G$1" pin="2"/>
+<pinref part="EN-3.3V" gate="G$1" pin="2"/>
 <wire x1="170.18" y1="-17.78" x2="170.18" y2="-22.86" width="0.1524" layer="91"/>
 <label x="170.18" y="-22.86" size="1.4224" layer="95" rot="R270" xref="yes"/>
@@
 <net name="ENABLE_SIGNAL" class="0">
 <segment>
-<pinref part="U$5" gate="G$1" pin="PIN2"/>
-<wire x1="180.34" y1="30.48" x2="180.34" y2="15.24" width="0.1524" layer="91"/>
-<label x="180.34" y="5.08" size="1.778" layer="95" rot="R90"/>
-</segment>
-<segment>
 <pinref part="U1" gate="G$1" pin="D27"/>
 <wire x1="-10.16" y1="-60.96" x2="-5.08" y2="-60.96" width="0.1524" layer="91"/>
 <label x="-5.08" y="-60.96" size="1.016" layer="95" xref="yes"/>
 </segment>
+<segment>
+<wire x1="185.42" y1="15.24" x2="185.42" y2="10.16" width="0.1524" layer="91"/>
+<label x="185.42" y="12.7" size="1.778" layer="95" rot="R90"/>
+<pinref part="3.3-BUZ1" gate="G$1" pin="1"/>
+</segment>
 </net>
 <net name="RX1_ESP" class="0">
@@
 </segment>
 <segment>
+<pinref part="GPS-TX-RX" gate="G$1" pin="2"/>
+<wire x1="-48.26" y1="88.9" x2="-48.26" y2="81.28" width="0.1524" layer="91"/>
+<label x="-48.26" y="81.28" size="1.4224" layer="95" rot="R270" xref="yes"/>
+</segment>
+</net>
+<net name="TX1_ESP" class="0">
+<segment>
+<pinref part="U1" gate="G$1" pin="D4"/>
+<wire x1="-40.64" y1="-53.34" x2="-45.72" y2="-53.34" width="0.1524" layer="91"/>
+<label x="-45.72" y="-53.34" size="1.016" layer="95" rot="R180" xref="yes"/>
+</segment>
+<segment>
 <pinref part="GPS-TX-RX" gate="G$1" pin="1"/>
 <wire x1="-50.8" y1="88.9" x2="-50.8" y2="81.28" width="0.1524" layer="91"/>
@@
 </segment>
 </net>
-<net name="TX1_ESP" class="0">
-<segment>
-<pinref part="U1" gate="G$1" pin="D4"/>
-<wire x1="-40.64" y1="-53.34" x2="-45.72" y2="-53.34" width="0.1524" layer="91"/>
-<label x="-45.72" y="-53.34" size="1.016" layer="95" rot="R180" xref="yes"/>
-</segment>
-<segment>
-<pinref part="GPS-TX-RX" gate="G$1" pin="2"/>
-<wire x1="-48.26" y1="88.9" x2="-48.26" y2="81.28" width="0.1524" layer="91"/>
-<label x="-48.26" y="81.28" size="1.4224" layer="95" rot="R270" xref="yes"/>
-</segment>
-</net>

Commit message: correções avionica e paraquedas
Parts:
- added GND, SK1-SK2: (no value), SparkFun-Connectors:CONN_022.54MM_SCREWTERM
Connections:
- new net SK1: SK1-SK2.1, U1.D25
- new net SK2: SK1-SK2.2, U1.D26
- net GND: now also GND.1, GND.2
Other:
- moved on the sheet: EN-3.3V, GPS-G-V, GPS-TX-RX, SKIB2-SKIB1
Changed lines of the file:
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@@
 <part name="GND-BAT" library="SparkFun-Connectors" deviceset="CONN_02" device="2.54MM_SCREWTERM"/>
 <part name="3.3-BUZ1" library="SparkFun-Connectors" deviceset="CONN_02" device="2.54MM_SCREWTERM"/>
+<part name="GND" library="SparkFun-Connectors" deviceset="CONN_02" device="2.54MM_SCREWTERM"/>
+<part name="SK1-SK2" library="SparkFun-Connectors" deviceset="CONN_02" device="2.54MM_SCREWTERM"/>
 </parts>
 <sheets>
@@
 <attribute name="VALUE" x="88.9" y="-78.74" size="1.778" layer="96"/>
 </instance>
-<instance part="GPS-TX-RX" gate="G$1" x="-50.8" y="96.52" smashed="yes" rot="R270">
-<attribute name="VALUE" x="-55.626" y="99.06" size="1.778" layer="96" font="vector" rot="R270"/>
-<attribute name="NAME" x="-45.212" y="99.06" size="1.778" layer="95" font="vector" rot="R270"/>
-</instance>
-<instance part="GPS-G-V" gate="G$1" x="-60.96" y="96.52" smashed="yes" rot="R270">
-<attribute name="VALUE" x="-65.786" y="99.06" size="1.778" layer="96" font="vector" rot="R270"/>
-<attribute name="NAME" x="-55.372" y="99.06" size="1.778" layer="95" font="vector" rot="R270"/>
-</instance>
-<instance part="EN-3.3V" gate="G$1" x="167.64" y="-10.16" smashed="yes" rot="R270">
-<attribute name="VALUE" x="162.814" y="-7.62" size="1.778" layer="96" font="vector" rot="R270"/>
-<attribute name="NAME" x="173.228" y="-7.62" size="1.778" layer="95" font="vector" rot="R270"/>
-</instance>
-<instance part="SKIB2-SKIB1" gate="G$1" x="154.94" y="-10.16" smashed="yes" rot="R270">
-<attribute name="VALUE" x="150.114" y="-7.62" size="1.778" layer="96" font="vector" rot="R270"/>
-<attribute name="NAME" x="160.528" y="-7.62" size="1.778" layer="95" font="vector" rot="R270"/>
+<instance part="GPS-TX-RX" gate="G$1" x="165.1" y="-15.24" smashed="yes" rot="R270">
+<attribute name="VALUE" x="160.274" y="-12.7" size="1.778" layer="96" font="vector" rot="R270"/>
+<attribute name="NAME" x="170.688" y="-12.7" size="1.778" layer="95" font="vector" rot="R270"/>
+</instance>
+<instance part="GPS-G-V" gate="G$1" x="154.94" y="-15.24" smashed="yes" rot="R270">
+<attribute name="VALUE" x="150.114" y="-12.7" size="1.778" layer="96" font="vector" rot="R270"/>
+<attribute name="NAME" x="160.528" y="-12.7" size="1.778" layer="95" font="vector" rot="R270"/>
+</instance>
+<instance part="EN-3.3V" gate="G$1" x="157.48" y="2.54" smashed="yes" rot="R90">
+<attribute name="VALUE" x="162.306" y="0" size="1.778" layer="96" font="vector" rot="R90"/>
+<attribute name="NAME" x="151.892" y="0" size="1.778" layer="95" font="vector" rot="R90"/>
+</instance>
+<instance part="SKIB2-SKIB1" gate="G$1" x="170.18" y="2.54" smashed="yes" rot="R90">
+<attribute name="VALUE" x="175.006" y="0" size="1.778" layer="96" font="vector" rot="R90"/>
+<attribute name="NAME" x="164.592" y="0" size="1.778" layer="95" font="vector" rot="R90"/>
 </instance>
 <instance part="GND-BAT" gate="G$1" x="167.64" y="93.98" smashed="yes" rot="R270">
@@
 <attribute name="VALUE" x="190.246" y="0" size="1.778" layer="96" font="vector" rot="R90"/>
 <attribute name="NAME" x="179.832" y="0" size="1.778" layer="95" font="vector" rot="R90"/>
+</instance>
+<instance part="GND" gate="G$1" x="200.66" y="2.54" smashed="yes" rot="R90">
+<attribute name="VALUE" x="205.486" y="0" size="1.778" layer="96" font="vector" rot="R90"/>
+<attribute name="NAME" x="195.072" y="0" size="1.778" layer="95" font="vector" rot="R90"/>
+</instance>
+<instance part="SK1-SK2" gate="G$1" x="210.82" y="2.54" smashed="yes" rot="R90">
+<attribute name="VALUE" x="215.646" y="0" size="1.778" layer="96" font="vector" rot="R90"/>
+<attribute name="NAME" x="205.232" y="0" size="1.778" layer="95" font="vector" rot="R90"/>
 </instance>
 </instances>
@@
 <segment>
 <pinref part="GPS-G-V" gate="G$1" pin="1"/>
-<wire x1="-60.96" y1="88.9" x2="-60.96" y2="81.28" width="0.1524" layer="91"/>
-<label x="-60.96" y="81.28" size="1.27" layer="95" rot="R270" xref="yes"/>
+<wire x1="154.94" y1="-22.86" x2="154.94" y2="-30.48" width="0.1524" layer="91"/>
+<label x="154.94" y="-30.48" size="1.27" layer="95" rot="R270" xref="yes"/>
+</segment>
+<segment>
+<pinref part="GND" gate="G$1" pin="2"/>
+<wire x1="198.12" y1="10.16" x2="198.12" y2="15.24" width="0.1524" layer="91"/>
+<pinref part="GND" gate="G$1" pin="1"/>
+<wire x1="198.12" y1="15.24" x2="200.66" y2="15.24" width="0.1524" layer="91"/>
+<wire x1="200.66" y1="15.24" x2="200.66" y2="10.16" width="0.1524" layer="91"/>
+<label x="198.12" y="12.7" size="1.778" layer="95" rot="R90"/>
 </segment>
 </net>
@@
 <segment>
 <pinref part="GPS-G-V" gate="G$1" pin="2"/>
-<wire x1="-58.42" y1="88.9" x2="-58.42" y2="81.28" width="0.1524" layer="91"/>
-<label x="-58.42" y="81.28" size="1.27" layer="95" rot="R270" xref="yes"/>
+<wire x1="157.48" y1="-22.86" x2="157.48" y2="-30.48" width="0.1524" layer="91"/>
+<label x="157.48" y="-30.48" size="1.27" layer="95" rot="R270" xref="yes"/>
 </segment>
 <segment>
 <pinref part="EN-3.3V" gate="G$1" pin="1"/>
-<wire x1="167.64" y1="-17.78" x2="167.64" y2="-22.86" width="0.1524" layer="91"/>
-<label x="167.64" y="-22.86" size="1.4224" layer="95" rot="R270" xref="yes"/>
+<wire x1="157.48" y1="10.16" x2="157.48" y2="15.24" width="0.1524" layer="91"/>
+<label x="157.48" y="15.24" size="1.4224" layer="95" rot="R90" xref="yes"/>
 </segment>
 <segment>
@@
 <segment>
 <pinref part="SKIB2-SKIB1" gate="G$1" pin="2"/>
-<wire x1="157.48" y1="-17.78" x2="157.48" y2="-22.86" width="0.1524" layer="91"/>
-<label x="157.48" y="-22.86" size="1.4224" layer="95" rot="R270" xref="yes"/>
+<wire x1="167.64" y1="10.16" x2="167.64" y2="15.24" width="0.1524" layer="91"/>
+<label x="167.64" y="15.24" size="1.4224" layer="95" rot="R90" xref="yes"/>
 </segment>
 </net>
@@
 <segment>
 <pinref part="SKIB2-SKIB1" gate="G$1" pin="1"/>
-<wire x1="154.94" y1="-17.78" x2="154.94" y2="-22.86" width="0.1524" layer="91"/>
-<label x="154.94" y="-22.86" size="1.4224" layer="95" rot="R270" xref="yes"/>
+<wire x1="170.18" y1="10.16" x2="170.18" y2="15.24" width="0.1524" layer="91"/>
+<label x="170.18" y="15.24" size="1.4224" layer="95" rot="R90" xref="yes"/>
 </segment>
 </net>
@@
 <segment>
 <pinref part="EN-3.3V" gate="G$1" pin="2"/>
-<wire x1="170.18" y1="-17.78" x2="170.18" y2="-22.86" width="0.1524" layer="91"/>
-<label x="170.18" y="-22.86" size="1.4224" layer="95" rot="R270" xref="yes"/>
+<wire x1="154.94" y1="10.16" x2="154.94" y2="15.24" width="0.1524" layer="91"/>
+<label x="154.94" y="15.24" size="1.4224" layer="95" rot="R90" xref="yes"/>
 </segment>
 </net>
@@
 <segment>
 <pinref part="GPS-TX-RX" gate="G$1" pin="2"/>
-<wire x1="-48.26" y1="88.9" x2="-48.26" y2="81.28" width="0.1524" layer="91"/>
-<label x="-48.26" y="81.28" size="1.4224" layer="95" rot="R270" xref="yes"/>
+<wire x1="167.64" y1="-22.86" x2="167.64" y2="-30.48" width="0.1524" layer="91"/>
+<label x="167.64" y="-30.48" size="1.4224" layer="95" rot="R270" xref="yes"/>
 </segment>
 </net>
@@
 <segment>
 <pinref part="GPS-TX-RX" gate="G$1" pin="1"/>
-<wire x1="-50.8" y1="88.9" x2="-50.8" y2="81.28" width="0.1524" layer="91"/>
-<label x="-50.8" y="81.28" size="1.4224" layer="95" rot="R270" xref="yes"/>
+<wire x1="165.1" y1="-22.86" x2="165.1" y2="-30.48" width="0.1524" layer="91"/>
+<label x="165.1" y="-30.48" size="1.4224" layer="95" rot="R270" xref="yes"/>
 </segment>
 </net>
@@
 </segment>
 </net>
+<net name="SK2" class="0">
+<segment>
+<pinref part="SK1-SK2" gate="G$1" pin="2"/>
+<wire x1="208.28" y1="10.16" x2="208.28" y2="15.24" width="0.1524" layer="91"/>
+<label x="208.28" y="12.7" size="1.778" layer="95" rot="R90"/>
+</segment>
+<segment>
+<pinref part="U1" gate="G$1" pin="D26"/>
+<wire x1="-10.16" y1="-58.42" x2="-5.08" y2="-58.42" width="0.1524" layer="91"/>
+<label x="-7.62" y="-58.42" size="1.778" layer="95"/>
+</segment>
+</net>
+<net name="SK1" class="0">
+<segment>
+<pinref part="SK1-SK2" gate="G$1" pin="1"/>
+<wire x1="210.82" y1="10.16" x2="210.82" y2="15.24" width="0.1524" layer="91"/>
+<label x="213.36" y="12.7" size="1.778" layer="95" rot="R90"/>
+</segment>
+<segment>
+<pinref part="U1" gate="G$1" pin="D25"/>
+<wire x1="-10.16" y1="-55.88" x2="-5.08" y2="-55.88" width="0.1524" layer="91"/>
+<label x="-7.62" y="-55.88" size="1.778" layer="95"/>
+</segment>
+</net>

Commit message: update
Parts:
- removed 3.3-BUZ1: (no value), SparkFun-Connectors:CONN_022.54MM_SCREWTERM
- added 3.3V-BUZ: (no value), SparkFun-Connectors:CONN_022.54MM_SCREWTERM
Connections:
- net BUZZER: now also 3.3V-BUZ.2; no longer EN-3.3V.2
- net ENABLE_SIGNAL: now also EN-3.3V.1; no longer 3.3-BUZ1.1
- net V_3V3: now also 3.3V-BUZ.1, EN-3.3V.2; no longer 3.3-BUZ1.2, EN-3.3V.1
Other:
- moved on the sheet: EN-3.3V
Changed lines of the file:
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@@
 <part name="GPS-TX-RX" library="SparkFun-Connectors" deviceset="CONN_02" device="2.54MM_SCREWTERM"/>
 <part name="GPS-G-V" library="SparkFun-Connectors" deviceset="CONN_02" device="2.54MM_SCREWTERM"/>
-<part name="EN-3.3V" library="SparkFun-Connectors" deviceset="CONN_02" device="2.54MM_SCREWTERM"/>
+<part name="3.3V-BUZ" library="SparkFun-Connectors" deviceset="CONN_02" device="2.54MM_SCREWTERM"/>
 <part name="SKIB2-SKIB1" library="SparkFun-Connectors" deviceset="CONN_02" device="2.54MM_SCREWTERM"/>
 <part name="GND-BAT" library="SparkFun-Connectors" deviceset="CONN_02" device="2.54MM_SCREWTERM"/>
-<part name="3.3-BUZ1" library="SparkFun-Connectors" deviceset="CONN_02" device="2.54MM_SCREWTERM"/>
+<part name="EN-3.3V" library="SparkFun-Connectors" deviceset="CONN_02" device="2.54MM_SCREWTERM"/>
 <part name="GND" library="SparkFun-Connectors" deviceset="CONN_02" device="2.54MM_SCREWTERM"/>
 <part name="SK1-SK2" library="SparkFun-Connectors" deviceset="CONN_02" device="2.54MM_SCREWTERM"/>
@@
 <attribute name="NAME" x="160.528" y="-12.7" size="1.778" layer="95" font="vector" rot="R270"/>
 </instance>
-<instance part="EN-3.3V" gate="G$1" x="157.48" y="2.54" smashed="yes" rot="R90">
+<instance part="3.3V-BUZ" gate="G$1" x="157.48" y="2.54" smashed="yes" rot="R90">
 <attribute name="VALUE" x="162.306" y="0" size="1.778" layer="96" font="vector" rot="R90"/>
 <attribute name="NAME" x="151.892" y="0" size="1.778" layer="95" font="vector" rot="R90"/>
@@
 <attribute name="NAME" x="173.228" y="96.52" size="1.778" layer="95" font="vector" rot="R270"/>
 </instance>
-<instance part="3.3-BUZ1" gate="G$1" x="185.42" y="2.54" smashed="yes" rot="R90">
+<instance part="EN-3.3V" gate="G$1" x="185.42" y="2.54" smashed="yes" rot="R90">
 <attribute name="VALUE" x="190.246" y="0" size="1.778" layer="96" font="vector" rot="R90"/>
 <attribute name="NAME" x="179.832" y="0" size="1.778" layer="95" font="vector" rot="R90"/>
@@
 </segment>
 <segment>
-<pinref part="EN-3.3V" gate="G$1" pin="1"/>
+<pinref part="3.3V-BUZ" gate="G$1" pin="1"/>
 <wire x1="157.48" y1="10.16" x2="157.48" y2="15.24" width="0.1524" layer="91"/>
 <label x="157.48" y="15.24" size="1.4224" layer="95" rot="R90" xref="yes"/>
 </segment>
 <segment>
-<pinref part="3.3-BUZ1" gate="G$1" pin="2"/>
+<pinref part="EN-3.3V" gate="G$1" pin="2"/>
 <wire x1="182.88" y1="10.16" x2="182.88" y2="15.24" width="0.1524" layer="91"/>
 <label x="180.34" y="12.7" size="1.778" layer="95" rot="R90"/>
@@
 </segment>
 <segment>
-<pinref part="EN-3.3V" gate="G$1" pin="2"/>
+<pinref part="3.3V-BUZ" gate="G$1" pin="2"/>
 <wire x1="154.94" y1="10.16" x2="154.94" y2="15.24" width="0.1524" layer="91"/>
 <label x="154.94" y="15.24" size="1.4224" layer="95" rot="R90" xref="yes"/>
@@
 <wire x1="185.42" y1="15.24" x2="185.42" y2="10.16" width="0.1524" layer="91"/>
 <label x="185.42" y="12.7" size="1.778" layer="95" rot="R90"/>
-<pinref part="3.3-BUZ1" gate="G$1" pin="1"/>
-</segment>
-</net>
+<pinref part="EN-3.3V" gate="G$1" pin="1"/>
+</segment>
+</net>
