File: Aviônica/Avionica 2.2/MODULO GPS.brd (EAGLE design)
At the start: 50 x 70.9 mm, 5 parts

Commit message: correções avionica e paraquedas
Changed lines of the file:
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@@
 <grid distance="0.000333" unitdist="inch" unit="inch" style="lines" multiple="1" display="yes" altdistance="0.1" altunitdist="mm" altunit="mm"/>
 <layers>
-<layer number="1" name="Top" color="4" fill="1" visible="no" active="yes"/>
+<layer number="1" name="Top" color="4" fill="1" visible="yes" active="yes"/>
 <layer number="2" name="Route2" color="16" fill="1" visible="no" active="no"/>
 <layer number="3" name="Route3" color="17" fill="1" visible="no" active="no"/>
@@
 <layer number="21" name="tPlace" color="7" fill="1" visible="yes" active="yes"/>
 <layer number="22" name="bPlace" color="7" fill="1" visible="yes" active="yes"/>
-<layer number="23" name="tOrigins" color="15" fill="1" visible="no" active="yes"/>
+<layer number="23" name="tOrigins" color="15" fill="1" visible="yes" active="yes"/>
 <layer number="24" name="bOrigins" color="15" fill="1" visible="yes" active="yes"/>
-<layer number="25" name="tNames" color="7" fill="1" visible="no" active="yes"/>
+<layer number="25" name="tNames" color="7" fill="1" visible="yes" active="yes"/>
 <layer number="26" name="bNames" color="7" fill="1" visible="yes" active="yes"/>
-<layer number="27" name="tValues" color="7" fill="1" visible="no" active="yes"/>
-<layer number="28" name="bValues" color="7" fill="1" visible="no" active="yes"/>
-<layer number="29" name="tStop" color="7" fill="3" visible="no" active="yes"/>
-<layer number="30" name="bStop" color="7" fill="6" visible="no" active="yes"/>
-<layer number="31" name="tCream" color="7" fill="4" visible="no" active="yes"/>
-<layer number="32" name="bCream" color="7" fill="5" visible="no" active="yes"/>
-<layer number="33" name="tFinish" color="6" fill="3" visible="no" active="yes"/>
-<layer number="34" name="bFinish" color="6" fill="6" visible="no" active="yes"/>
-<layer number="35" name="tGlue" color="7" fill="4" visible="no" active="yes"/>
-<layer number="36" name="bGlue" color="7" fill="5" visible="no" active="yes"/>
-<layer number="37" name="tTest" color="7" fill="1" visible="no" active="yes"/>
-<layer number="38" name="bTest" color="7" fill="1" visible="no" active="yes"/>
-<layer number="39" name="tKeepout" color="4" fill="11" visible="no" active="yes"/>
+<layer number="27" name="tValues" color="7" fill="1" visible="yes" active="yes"/>
+<layer number="28" name="bValues" color="7" fill="1" visible="yes" active="yes"/>
+<layer number="29" name="tStop" color="7" fill="3" visible="yes" active="yes"/>
+<layer number="30" name="bStop" color="7" fill="6" visible="yes" active="yes"/>
+<layer number="31" name="tCream" color="7" fill="4" visible="yes" active="yes"/>
+<layer number="32" name="bCream" color="7" fill="5" visible="yes" active="yes"/>
+<layer number="33" name="tFinish" color="6" fill="3" visible="yes" active="yes"/>
+<layer number="34" name="bFinish" color="6" fill="6" visible="yes" active="yes"/>
+<layer number="35" name="tGlue" color="7" fill="4" visible="yes" active="yes"/>
+<layer number="36" name="bGlue" color="7" fill="5" visible="yes" active="yes"/>
+<layer number="37" name="tTest" color="7" fill="1" visible="yes" active="yes"/>
+<layer number="38" name="bTest" color="7" fill="1" visible="yes" active="yes"/>
+<layer number="39" name="tKeepout" color="4" fill="11" visible="yes" active="yes"/>
 <layer number="40" name="bKeepout" color="1" fill="11" visible="yes" active="yes"/>
-<layer number="41" name="tRestrict" color="4" fill="10" visible="no" active="yes"/>
+<layer number="41" name="tRestrict" color="4" fill="10" visible="yes" active="yes"/>
 <layer number="42" name="bRestrict" color="1" fill="10" visible="yes" active="yes"/>
-<layer number="43" name="vRestrict" color="2" fill="10" visible="no" active="yes"/>
-<layer number="44" name="Drills" color="7" fill="1" visible="no" active="yes"/>
-<layer number="45" name="Holes" color="7" fill="1" visible="no" active="yes"/>
-<layer number="46" name="Milling" color="3" fill="1" visible="no" active="yes"/>
-<layer number="47" name="Measures" color="7" fill="1" visible="no" active="yes"/>
-<layer number="48" name="Document" color="7" fill="1" visible="no" active="yes"/>
-<layer number="49" name="Reference" color="7" fill="1" visible="no" active="yes"/>
-<layer number="50" name="dxf" color="7" fill="1" visible="no" active="yes"/>
-<layer number="51" name="tDocu" color="7" fill="1" visible="no" active="yes"/>
+<layer number="43" name="vRestrict" color="2" fill="10" visible="yes" active="yes"/>
+<layer number="44" name="Drills" color="7" fill="1" visible="yes" active="yes"/>
+<layer number="45" name="Holes" color="7" fill="1" visible="yes" active="yes"/>
+<layer number="46" name="Milling" color="3" fill="1" visible="yes" active="yes"/>
+<layer number="47" name="Measures" color="7" fill="1" visible="yes" active="yes"/>
+<layer number="48" name="Document" color="7" fill="1" visible="yes" active="yes"/>
+<layer number="49" name="Reference" color="7" fill="1" visible="yes" active="yes"/>
+<layer number="50" name="dxf" color="7" fill="1" visible="yes" active="yes"/>
+<layer number="51" name="tDocu" color="7" fill="1" visible="yes" active="yes"/>
 <layer number="52" name="bDocu" color="7" fill="1" visible="yes" active="yes"/>
 <layer number="53" name="tGND_GNDA" color="7" fill="9" visible="no" active="no"/>
@@
 <layer number="196" name="mValues" color="7" fill="1" visible="no" active="no"/>
 <layer number="199" name="Contour" color="7" fill="1" visible="no" active="no"/>
-<layer number="200" name="200bmp" color="1" fill="10" visible="no" active="yes"/>
+<layer number="200" name="200bmp" color="1" fill="10" visible="yes" active="yes"/>
 <layer number="201" name="201bmp" color="2" fill="10" visible="no" active="no"/>
 <layer number="202" name="202bmp" color="3" fill="10" visible="no" active="no"/>
@@
 <element name="U$3" library="CRD" library_urn="urn:adsk.eagle:library:39051337" package="GPS_MODULE_FOOTPRINT" package3d_urn="urn:adsk.eagle:package:39608400/4" value="GPS_MODULE" x="89.549" y="38.812" smashed="yes" rot="R90"/>
 <element name="TX-RX" library="SparkFun-Connectors" package="1X02_2.54_SCREWTERM" value="" x="113.5136" y="36.8864" smashed="yes" rot="R90">
-<attribute name="NAME" x="117.339" y="36.4784" size="0.8128" layer="26" font="vector" ratio="20" rot="MR90"/>
+<attribute name="NAME" x="118.201734375" y="36.436109375" size="0.8128" layer="25" font="vector" ratio="20" rot="R90"/>
 <attribute name="VALUE" x="117.5776" y="35.6164" size="0.6096" layer="27" font="vector" ratio="20" rot="R90"/>
 </element>

Commit message: update
Parts:
- removed TX-RX: (no value), SparkFun-Connectors:1X02_2.54_SCREWTERM
- added RX-TX: (no value), SparkFun-Connectors:1X02_2.54_SCREWTERM
- moved GND-3.3V 16.1 mm to (113.8, 28.5)
- moved EN-3.3V 4.77 mm to (113.7, 20.6)
Connections:
- net GND: now also GND-3.3V.P2; no longer GND-3.3V.P1
- net RX1_ESP: now also RX-TX.P2; no longer TX-RX.P2
- net TX1_ESP: now also RX-TX.P1; no longer TX-RX.P1
- net V_3V3: now also GND-3.3V.P1; no longer GND-3.3V.P2
Routing:
- net RX1_ESP: track 7.64 -> 33.2 mm
- net V_3V3: track 56.4 -> 79.0 mm
- net TX1_ESP: track 7.64 -> 29.1 mm
- net ENABLE_SIGNAL: track 27.8 -> 27.1 mm
Changed lines of the file:
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@@
 <setting verticaltext="up"/>
 </settings>
-<grid distance="0.000333" unitdist="inch" unit="inch" style="lines" multiple="1" display="yes" altdistance="0.1" altunitdist="mm" altunit="mm"/>
+<grid distance="0.000333" unitdist="inch" unit="mm" style="lines" multiple="1" display="yes" altdistance="0.1" altunitdist="mm" altunit="mm"/>
 <layers>
 <layer number="1" name="Top" color="4" fill="1" visible="yes" active="yes"/>
@@
 <elements>
 <element name="U$3" library="CRD" library_urn="urn:adsk.eagle:library:39051337" package="GPS_MODULE_FOOTPRINT" package3d_urn="urn:adsk.eagle:package:39608400/4" value="GPS_MODULE" x="89.549" y="38.812" smashed="yes" rot="R90"/>
-<element name="TX-RX" library="SparkFun-Connectors" package="1X02_2.54_SCREWTERM" value="" x="113.5136" y="36.8864" smashed="yes" rot="R90">
-<attribute name="NAME" x="118.201734375" y="36.436109375" size="0.8128" layer="25" font="vector" ratio="20" rot="R90"/>
-<attribute name="VALUE" x="117.5776" y="35.6164" size="0.6096" layer="27" font="vector" ratio="20" rot="R90"/>
+<element name="RX-TX" library="SparkFun-Connectors" package="1X02_2.54_SCREWTERM" value="" x="113.62355625" y="12.4252875" smashed="yes" rot="R90">
+<attribute name="NAME" x="118.311690625" y="11.974996875" size="0.8128" layer="25" font="vector" ratio="20" rot="R90"/>
+<attribute name="VALUE" x="117.68755625" y="11.1552875" size="0.6096" layer="27" font="vector" ratio="20" rot="R90"/>
 </element>
-<element name="GND-3.3V" library="SparkFun-Connectors" package="1X02_2.54_SCREWTERM" value="" x="113.568" y="44.6304" smashed="yes" rot="R90">
-<attribute name="NAME" x="118.0346" y="43.2572" size="0.8128" layer="25" font="vector" ratio="20" rot="R90"/>
-<attribute name="VALUE" x="117.632" y="43.3604" size="0.6096" layer="27" font="vector" ratio="20" rot="R90"/>
+<element name="GND-3.3V" library="SparkFun-Connectors" package="1X02_2.54_SCREWTERM" value="" x="113.754078125" y="28.542903125" smashed="yes" rot="R90">
+<attribute name="NAME" x="118.220678125" y="27.169703125" size="0.8128" layer="25" font="vector" ratio="20" rot="R90"/>
+<attribute name="VALUE" x="117.818078125" y="27.272903125" size="0.6096" layer="27" font="vector" ratio="20" rot="R90"/>
 </element>
 <element name="U$1" library="CRD" library_urn="urn:adsk.eagle:library:39051337" package="SWITCH_ALAVANCA_FOOTPRINT" value="SWITCH_ALAVANCA" x="92.51" y="20.58" smashed="yes"/>
-<element name="EN-3.3V" library="SparkFun-Connectors" package="1X02_2.54_SCREWTERM" value="" x="113.81" y="15.87" smashed="yes" rot="R90">
-<attribute name="NAME" x="118.101" y="15.22" size="0.6096" layer="25" font="vector" ratio="20" rot="R90"/>
-<attribute name="VALUE" x="117.874" y="14.6" size="0.6096" layer="27" font="vector" ratio="20" rot="R90"/>
+<element name="EN-3.3V" library="SparkFun-Connectors" package="1X02_2.54_SCREWTERM" value="" x="113.674675" y="20.640428125" smashed="yes" rot="R90">
+<attribute name="NAME" x="117.965675" y="19.990428125" size="0.8128" layer="25" font="vector" ratio="20" rot="R90"/>
+<attribute name="VALUE" x="117.738675" y="19.370428125" size="0.6096" layer="27" font="vector" ratio="20" rot="R90"/>
 </element>
 </elements>
@@
 </polygon>
 <contactref element="U$1" pad="PIN1"/>
-<contactref element="GND-3.3V" pad="P1"/>
 <via x="113.8" y="53.45" extent="1-16" drill="0.35"/>
 <via x="73.63" y="54.52" extent="1-16" drill="0.35"/>
@@
 <via x="82.14" y="8.9" extent="1-16" drill="0.35"/>
 <via x="103.13" y="46.71" extent="1-16" drill="0.35"/>
-<via x="114.69" y="29.11" extent="1-16" drill="0.35"/>
-<via x="103.13" y="14.29" extent="1-16" drill="0.35"/>
+<via x="110.59623125" y="50.5515375" extent="1-16" drill="0.35"/>
+<via x="102.0981" y="16.522965625" extent="1-16" drill="0.35"/>
+<contactref element="GND-3.3V" pad="P2"/>
+<via x="105.253840625" y="28.394178125" extent="1-16" drill="0.35"/>
+<via x="105.77825" y="31.819746875" extent="1-16" drill="0.35"/>
+<via x="113.923496875" y="26.059715625" extent="1-16" drill="0.35"/>
+<via x="111.9019875" y="26.059715625" extent="1-16" drill="0.35"/>
 </signal>
 <signal name="V_3V3">
@@
 <contactref element="U$1" pad="PIN3"/>
 <contactref element="EN-3.3V" pad="P1"/>
-<wire x1="113.81" y1="18.41" x2="96.078" y2="18.41" width="1.27" layer="16"/>
-<wire x1="96.078" y1="18.41" x2="95.708" y2="18.04" width="1.27" layer="16"/>
-<contactref element="GND-3.3V" pad="P2"/>
-<wire x1="106.059" y1="42.422" x2="108.2674" y2="44.6304" width="1.27" layer="16"/>
-<wire x1="108.2674" y1="44.6304" x2="113.568" y2="44.6304" width="1.27" layer="16"/>
-<wire x1="95.708" y1="18.04" x2="100.63" y2="22.962" width="1.27" layer="16"/>
-<wire x1="104.342" y1="42.422" x2="106.059" y2="42.422" width="1.27" layer="16"/>
-<wire x1="100.63" y1="22.962" x2="100.63" y2="38.71" width="1.27" layer="16"/>
-<wire x1="100.63" y1="38.71" x2="104.342" y2="42.422" width="1.27" layer="16"/>
+<contactref element="GND-3.3V" pad="P1"/>
+<wire x1="106.059" y1="42.422" x2="106.448" y2="42.033" width="1.27" layer="16"/>
+<wire x1="106.448" y1="42.033" x2="108.57919375" y2="42.033" width="1.27" layer="16"/>
+<wire x1="108.57919375" y1="42.033" x2="113.754078125" y2="36.858115625" width="1.27" layer="16"/>
+<wire x1="113.754078125" y1="36.858115625" x2="113.754078125" y2="31.082903125" width="1.27" layer="16"/>
+<wire x1="113.754078125" y1="31.082903125" x2="115.0155875" y2="31.082903125" width="1.27" layer="16"/>
+<wire x1="115.0155875" y1="31.082903125" x2="117.1376125" y2="28.960878125" width="1.27" layer="16"/>
+<wire x1="117.1376125" y1="28.960878125" x2="117.1376125" y2="24.03820625" width="1.27" layer="16"/>
+<wire x1="117.1376125" y1="24.03820625" x2="116.19029375" y2="23.0908875" width="1.27" layer="16"/>
+<wire x1="116.19029375" y1="23.0908875" x2="113.764215625" y2="23.0908875" width="1.27" layer="16"/>
+<wire x1="113.764215625" y1="23.0908875" x2="113.674675" y2="23.180428125" width="1.27" layer="16"/>
+<wire x1="95.708" y1="18.04" x2="100.848428125" y2="23.180428125" width="1.27" layer="1"/>
+<wire x1="100.848428125" y1="23.180428125" x2="113.674675" y2="23.180428125" width="1.27" layer="1"/>
+<wire x1="95.708" y1="18.04" x2="95.708" y2="34.36913125" width="1.27" layer="16"/>
+<wire x1="103.76086875" y1="42.422" x2="106.059" y2="42.422" width="1.27" layer="16"/>
+<wire x1="95.708" y1="34.36913125" x2="103.76086875" y2="42.422" width="1.27" layer="16"/>
 </signal>
 <signal name="RX1_ESP">
 <contactref element="U$3" pad="TX"/>
-<contactref element="TX-RX" pad="P2"/>
-<wire x1="106.059" y1="37.342" x2="106.481" y2="36.92" width="1.27" layer="16"/>
-<wire x1="113.48" y1="36.92" x2="113.5136" y2="36.8864" width="1.27" layer="16"/>
-<wire x1="106.481" y1="36.92" x2="113.48" y2="36.92" width="1.27" layer="16"/>
+<contactref element="RX-TX" pad="P2"/>
+<wire x1="113.62355625" y1="12.4252875" x2="113.5222125" y2="12.52663125" width="1" layer="16"/>
+<wire x1="113.5222125" y1="12.52663125" x2="109.08098125" y2="12.52663125" width="1" layer="16"/>
+<wire x1="109.08098125" y1="12.52663125" x2="103.333828125" y2="18.273784375" width="1" layer="16"/>
+<wire x1="103.333828125" y1="18.273784375" x2="103.333828125" y2="35.0846125" width="1" layer="16"/>
+<wire x1="103.333828125" y1="35.0846125" x2="105.591215625" y2="37.342" width="1" layer="16"/>
+<wire x1="105.591215625" y1="37.342" x2="106.059" y2="37.342" width="1" layer="16"/>
 </signal>
 <signal name="TX1_ESP">
 <contactref element="U$3" pad="RX"/>
-<contactref element="TX-RX" pad="P1"/>
-<wire x1="106.059" y1="39.882" x2="113.058" y2="39.882" width="1.27" layer="16"/>
-<wire x1="113.058" y1="39.882" x2="113.5136" y2="39.4264" width="1.27" layer="16"/>
+<contactref element="RX-TX" pad="P1"/>
+<wire x1="113.62355625" y1="14.9652875" x2="108.916240625" y2="19.672603125" width="1" layer="16"/>
+<wire x1="108.98390625" y1="31.675959375" x2="108.98390625" y2="38.586309375" width="1" layer="16"/>
+<wire x1="108.98390625" y1="38.586309375" x2="107.688215625" y2="39.882" width="1" layer="16"/>
+<wire x1="107.688215625" y1="39.882" x2="106.059" y2="39.882" width="1" layer="16"/>
+<wire x1="108.916240625" y1="19.672603125" x2="108.916240625" y2="31.60829375" width="1" layer="16"/>
+<wire x1="108.916240625" y1="31.60829375" x2="108.98390625" y2="31.675959375" width="1" layer="16"/>
 </signal>
 <signal name="ANTENNA">
@@
 <contactref element="U$1" pad="PIN2"/>
 <contactref element="EN-3.3V" pad="P2"/>
-<wire x1="109.65" y1="11.71" x2="95.23" y2="11.71" width="1.27" layer="16"/>
-<wire x1="109.65" y1="11.71" x2="113.81" y2="15.87" width="1.27" layer="16"/>
-<wire x1="92.458" y1="14.482" x2="92.458" y2="18.04" width="1.27" layer="16"/>
-<wire x1="95.23" y1="11.71" x2="92.458" y2="14.482" width="1.27" layer="16"/>
+<wire x1="103.9959875" y1="20.640428125" x2="113.674675" y2="20.640428125" width="1.27" layer="1"/>
+<wire x1="103.9959875" y1="20.640428125" x2="97.08321875" y2="13.727659375" width="1.27" layer="1"/>
+<wire x1="97.08321875" y1="13.727659375" x2="94.604965625" y2="13.727659375" width="1.27" layer="1"/>
+<wire x1="92.458" y1="15.874625" x2="92.458" y2="18.04" width="1.27" layer="1"/>
+<wire x1="94.604965625" y1="13.727659375" x2="92.458" y2="15.874625" width="1.27" layer="1"/>
 </signal>
 </signals>
