File: Aviônica/Avionica 2.2/MODULO GPS.sch (EAGLE design)
At the start: 12 parts, among them J1 MICRO-SD-PUSH-PUSH-EXT-PIN, U1 ESP32-DEVKIT-V1

Commit message: Atualização-avionica
Parts:
- removed 3.3-BUZ, 3.3-BUZ1, GND-BAT, GPS-G-V, GPS-TX-RX, SKIB2-SKIB1: (no value), SparkFun-Connectors:CONN_022.54MM_SCREWTERM
- removed J1: MICRO-SD-PUSH-PUSH-EXT-PIN, SparkFun-Connectors:MICRO-SD-PUSH-PUSH-EXT-PIN
- removed U$11: SWITCH_3PIN, CRD:SWITCH_3PIN
- removed U$2: E22-400T30D, CRD:E22-400T30D
- removed U$4: BMP280V1, CRD:BMP280V1
- removed U$6: MPU6050V1, CRD:MPU6050V1
- removed U1: ESP32-DEVKIT-V1, ESP32-DEVKIT-V1:ESP32-DEVKIT-V1
- added EN-3.3V, GND-3.3V, TX-RX: (no value), SparkFun-Connectors:CONN_022.54MM_SCREWTERM
- added U$1: SWITCH_ALAVANCA, CRD:SWITCH_ALAVANCA
- added U$3: GPS_MODULE, CRD:GPS_MODULE
Connections:
- removed net BUZZER: 3.3-BUZ.2, U1.D14
- removed net CS: J1.DAT3/!CS!, U1.D5
- removed net M0: U$2.M0, U1.D35
- removed net M1: U$2.M1, U1.D34
- removed net MISO: J1.DAT0/SDO, U1.D19
- removed net MOSI: J1.CMD/SDI, U1.D23
- removed net N$3: U$2.AUX
- removed net N$4: U$11.1
- removed net RX2_ESP: U$2.TXD, U1.RX2
- removed net SCK: J1.CLK/SCK, U1.D18
- removed net SCL: U$4.SCL, U$6.SCL, U1.D22
- removed net SDA: U$4.SDA, U$6.SDA, U1.D21
- removed net SKIB1: SKIB2-SKIB1.2, U1.D13
- removed net SKIB2: SKIB2-SKIB1.1, U1.D12
- removed net TX2_ESP: U$2.RXD, U1.TX2
- removed net V_BATTERY: GND-BAT.1, U$11.2
- removed net V_IN: U$11.3, U$2.VCC, U1.VIN
- net ENABLE_SIGNAL: now also EN-3.3V.2, U$1.PIN2; no longer 3.3-BUZ1.1, U1.D27
- net GND: now also GND-3.3V.1, U$1.PIN1, U$3.GND; no longer GND-BAT.2, GPS-G-V.1, J1.GND, U$2.GND, U$4.GND, U$6.GND, U1.GND
- net RX1_ESP: now also TX-RX.2, U$3.TX; no longer GPS-TX-RX.1, U1.D15
- net TX1_ESP: now also TX-RX.1, U$3.RX; no longer GPS-TX-RX.2, U1.D4
- net V_3V3: now also EN-3.3V.1, GND-3.3V.2, U$1.PIN3, U$3.VCC; no longer 3.3-BUZ.1, 3.3-BUZ1.2, GPS-G-V.2, J1.VCC, U$4.VCC, U$6.VCC, U1.3V3
Other:
- note removed: "# Observações: LoRa: Supports 3.3V~5.5V power supply, power supply over 5V can guarantee the best performance."
- note removed: "-> Passar por um elevador de tensão 5.0V ->"
- note removed: "Alimentação ESP32: A alimentação dessa placa pode ser feita através do próprio conector USB (5,0V) ou então através do pino 5V ou VIN , com uma alimentação regulada de 5,0V. Apesar do Regulador AMS1117 aceitar até 12V na entrada, recomendo que, se for alimentar a placa através desse pino, use sempre uma fonte regulada de 5V, pois assim nunca sobre-aquecerá o mesmo ! Evitando um possível defeito n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"

Commit message: update
Parts:
- renumbered TX-RX to RX-TX
Connections:
- net GND: now also GND-3.3V.2; no longer GND-3.3V.1
- net V_3V3: now also GND-3.3V.1; no longer GND-3.3V.2
Changed lines of the file:
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@@
 <part name="U$3" library="CRD" library_urn="urn:adsk.eagle:library:39051337" deviceset="GPS_MODULE" device="" package3d_urn="urn:adsk.eagle:package:39608400/4"/>
 <part name="GND3" library="supply1" library_urn="urn:adsk.eagle:library:371" deviceset="GND" device=""/>
-<part name="TX-RX" library="SparkFun-Connectors" deviceset="CONN_02" device="2.54MM_SCREWTERM"/>
+<part name="RX-TX" library="SparkFun-Connectors" deviceset="CONN_02" device="2.54MM_SCREWTERM"/>
 <part name="GND-3.3V" library="SparkFun-Connectors" deviceset="CONN_02" device="2.54MM_SCREWTERM"/>
 <part name="GND1" library="supply1" library_urn="urn:adsk.eagle:library:371" deviceset="GND" device=""/>
@@
 <attribute name="VALUE" x="-68.46094375" y="32.771934375" size="1.778" layer="96"/>
 </instance>
-<instance part="TX-RX" gate="G$1" x="-55.88" y="10.16" smashed="yes" rot="R90">
+<instance part="RX-TX" gate="G$1" x="-55.88" y="10.16" smashed="yes" rot="R90">
 <attribute name="VALUE" x="-51.054" y="7.62" size="1.778" layer="96" font="vector" rot="R90"/>
 <attribute name="NAME" x="-61.468" y="7.62" size="1.778" layer="95" font="vector" rot="R90"/>
@@
 <attribute name="NAME" x="-30.48" y="24.892" size="1.778" layer="95" font="vector" rot="R180"/>
 </instance>
-<instance part="GND1" gate="1" x="-40.75905625" y="38.348065625" smashed="yes" rot="R180">
-<attribute name="VALUE" x="-38.21905625" y="40.888065625" size="1.778" layer="96" rot="R180"/>
+<instance part="GND1" gate="1" x="-43.06094375" y="17.531934375" smashed="yes">
+<attribute name="VALUE" x="-45.60094375" y="14.991934375" size="1.778" layer="96"/>
 </instance>
 <instance part="U$1" gate="G$1" x="15.24" y="60.96" smashed="yes"/>
@@
 </segment>
 <segment>
+<pinref part="GND-3.3V" gate="G$1" pin="2"/>
 <pinref part="GND1" gate="1" pin="GND"/>
-<pinref part="GND-3.3V" gate="G$1" pin="1"/>
-<wire x1="-40.75905625" y1="35.808065625" x2="-40.64" y2="35.808065625" width="0.1524" layer="91"/>
-<wire x1="-40.64" y1="35.808065625" x2="-40.64" y2="30.48" width="0.1524" layer="91"/>
+<wire x1="-40.64" y1="27.94" x2="-43.06094375" y2="27.94" width="0.1524" layer="91"/>
+<wire x1="-43.06094375" y1="27.94" x2="-43.06094375" y2="20.071934375" width="0.1524" layer="91"/>
 </segment>
 </net>
@@
 <pinref part="U$3" gate="G$1" pin="VCC"/>
 <label x="-48.26" y="27.94" size="1.778" layer="95" rot="R90"/>
-<wire x1="-48.26" y1="43.18" x2="-48.26" y2="27.94" width="0.1524" layer="91"/>
-<pinref part="GND-3.3V" gate="G$1" pin="2"/>
-<wire x1="-40.64" y1="27.94" x2="-48.26" y2="27.94" width="0.1524" layer="91"/>
+<wire x1="-48.26" y1="43.18" x2="-48.26" y2="30.48" width="0.1524" layer="91"/>
+<pinref part="GND-3.3V" gate="G$1" pin="1"/>
+<wire x1="-48.26" y1="30.48" x2="-48.26" y2="27.94" width="0.1524" layer="91"/>
+<wire x1="-40.64" y1="30.48" x2="-48.26" y2="30.48" width="0.1524" layer="91"/>
+<junction x="-48.26" y="30.48"/>
 </segment>
 <segment>
@@
 <label x="-58.42" y="25.4" size="1.778" layer="95" rot="R90"/>
 <wire x1="-58.42" y1="17.78" x2="-58.42" y2="43.18" width="0.1524" layer="91"/>
-<pinref part="TX-RX" gate="G$1" pin="2"/>
+<pinref part="RX-TX" gate="G$1" pin="2"/>
 </segment>
 </net>
@@
 <label x="-53.34" y="25.4" size="1.778" layer="95" rot="R90"/>
 <wire x1="-53.34" y1="17.78" x2="-53.34" y2="43.18" width="0.1524" layer="91"/>
-<pinref part="TX-RX" gate="G$1" pin="1"/>
+<pinref part="RX-TX" gate="G$1" pin="1"/>
 <wire x1="-55.88" y1="17.78" x2="-53.34" y2="17.78" width="0.1524" layer="91"/>
 </segment>
