File: Paraquedas/Paraquedas 2.1/Esquema.sch (EAGLE design)
At the start: 20 parts, among them Q1 IRF540, Q2 IRF540, Q3 IRF540

Commit message: Message
Parts:
- removed LED3: 5mm, led:LED5MM
- removed R8: 220, rcl:R-EU_0207/10
- added LED2: 5mm, led:LED5MM
- added R7: 1k, rcl:R-EU_0207/10
- R1, R5: value 220 -> 1k
Connections:
- removed net N$3 (its old number): LED3.A, R8.2
- new net N$1: LED2.A, R7.2
- net GND: now also LED2.C; no longer LED3.C
- net SINAL_SKIB1: no longer R5.1
- net SINAL_SKIB2: no longer R8.1
- net SKIB1: now also U$2.1; no longer U$2.2
- net SKIB1_CONECTOR: now also R5.1
- net SKIB2: now also U$2.2; no longer U$2.1
- net SKIB2_CONECTOR: now also R7.1
Other:
- moved on the sheet: LED1, R5

Commit message: Update paraquedas
Parts:
- renumbered LED1 to LSKIB1, LED2 to LSKIB2, OK1 to GND
Changed lines of the file:
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@@
 <drawing>
 <settings>
-<setting alwaysvectorfont="yes"/>
+<setting alwaysvectorfont="no"/>
 <setting verticaltext="up"/>
 </settings>
@@
 <part name="GND3" library="supply1" library_urn="urn:adsk.eagle:library:371" deviceset="GND" device=""/>
 <part name="GND4" library="supply1" library_urn="urn:adsk.eagle:library:371" deviceset="GND" device=""/>
-<part name="OK1" library="optocoupler" library_urn="urn:adsk.eagle:library:320" deviceset="PC817" device="" package3d_urn="urn:adsk.eagle:package:21938/1"/>
+<part name="GND" library="optocoupler" library_urn="urn:adsk.eagle:library:320" deviceset="PC817" device="" package3d_urn="urn:adsk.eagle:package:21938/1"/>
 <part name="R1" library="rcl" library_urn="urn:adsk.eagle:library:334" deviceset="R-EU_" device="0207/10" package3d_urn="urn:adsk.eagle:package:23491/2" value="1k"/>
 <part name="R5" library="rcl" library_urn="urn:adsk.eagle:library:334" deviceset="R-EU_" device="0207/10" package3d_urn="urn:adsk.eagle:package:23491/2" value="1k"/>
-<part name="LED1" library="led" library_urn="urn:adsk.eagle:library:259" deviceset="LED" device="5MM" package3d_urn="urn:adsk.eagle:package:15799/2" value="5mm"/>
+<part name="LSKIB1" library="led" library_urn="urn:adsk.eagle:library:259" deviceset="LED" device="5MM" package3d_urn="urn:adsk.eagle:package:15799/2" value="5mm"/>
 <part name="GND5" library="supply1" library_urn="urn:adsk.eagle:library:371" deviceset="GND" device=""/>
 <part name="GND7" library="supply1" library_urn="urn:adsk.eagle:library:371" deviceset="GND" device=""/>
@@
 <part name="R6" library="rcl" library_urn="urn:adsk.eagle:library:334" deviceset="R-EU_" device="0207/10" package3d_urn="urn:adsk.eagle:package:23491/2" value="1k"/>
 <part name="R7" library="rcl" library_urn="urn:adsk.eagle:library:334" deviceset="R-EU_" device="0207/10" package3d_urn="urn:adsk.eagle:package:23491/2" value="1k"/>
-<part name="LED2" library="led" library_urn="urn:adsk.eagle:library:259" deviceset="LED" device="5MM" package3d_urn="urn:adsk.eagle:package:15799/2" value="5mm"/>
+<part name="LSKIB2" library="led" library_urn="urn:adsk.eagle:library:259" deviceset="LED" device="5MM" package3d_urn="urn:adsk.eagle:package:15799/2" value="5mm"/>
 <part name="GND9" library="supply1" library_urn="urn:adsk.eagle:library:371" deviceset="GND" device=""/>
 <part name="GND11" library="supply1" library_urn="urn:adsk.eagle:library:371" deviceset="GND" device=""/>
@@
 <attribute name="VALUE" x="50.8" y="-78.74" size="1.778" layer="96"/>
 </instance>
-<instance part="OK1" gate="A" x="137.16" y="40.64" smashed="yes">
+<instance part="GND" gate="A" x="137.16" y="40.64" smashed="yes">
 <attribute name="NAME" x="130.175" y="46.355" size="1.778" layer="95"/>
 <attribute name="VALUE" x="130.175" y="33.02" size="1.778" layer="96"/>
@@
 <attribute name="VALUE" x="98.298" y="36.83" size="1.778" layer="96" rot="R270"/>
 </instance>
-<instance part="LED1" gate="G$1" x="106.68" y="22.86" smashed="yes" rot="R90">
+<instance part="LSKIB1" gate="G$1" x="106.68" y="22.86" smashed="yes" rot="R90">
 <attribute name="NAME" x="111.252" y="26.416" size="1.778" layer="95" rot="R180"/>
 <attribute name="VALUE" x="111.252" y="28.575" size="1.778" layer="96" rot="R180"/>
@@
 <attribute name="VALUE" x="98.298" y="-6.35" size="1.778" layer="96" rot="R270"/>
 </instance>
-<instance part="LED2" gate="G$1" x="106.68" y="-20.32" smashed="yes" rot="R90">
+<instance part="LSKIB2" gate="G$1" x="106.68" y="-20.32" smashed="yes" rot="R90">
 <attribute name="NAME" x="111.252" y="-16.764" size="1.778" layer="95" rot="R180"/>
 <attribute name="VALUE" x="111.252" y="-14.605" size="1.778" layer="96" rot="R180"/>
@@
 </segment>
 <segment>
-<pinref part="LED1" gate="G$1" pin="C"/>
+<pinref part="LSKIB1" gate="G$1" pin="C"/>
 <pinref part="GND7" gate="1" pin="GND"/>
 <wire x1="111.76" y1="22.86" x2="116.84" y2="22.86" width="0.1524" layer="91"/>
@@
 <pinref part="GND5" gate="1" pin="GND"/>
 <wire x1="124.46" y1="30.48" x2="124.46" y2="38.1" width="0.1524" layer="91"/>
-<pinref part="OK1" gate="A" pin="C"/>
+<pinref part="GND" gate="A" pin="C"/>
 <wire x1="124.46" y1="38.1" x2="127" y2="38.1" width="0.1524" layer="91"/>
 </segment>
 <segment>
-<pinref part="LED2" gate="G$1" pin="C"/>
+<pinref part="LSKIB2" gate="G$1" pin="C"/>
 <pinref part="GND11" gate="1" pin="GND"/>
 <wire x1="111.76" y1="-20.32" x2="116.84" y2="-20.32" width="0.1524" layer="91"/>
@@
 <pinref part="R5" gate="G$1" pin="2"/>
 <wire x1="101.6" y1="27.94" x2="101.6" y2="22.86" width="0.1524" layer="91"/>
-<pinref part="LED1" gate="G$1" pin="A"/>
+<pinref part="LSKIB1" gate="G$1" pin="A"/>
 <wire x1="101.6" y1="22.86" x2="104.14" y2="22.86" width="0.1524" layer="91"/>
 </segment>
@@
 <segment>
 <pinref part="R1" gate="G$1" pin="1"/>
-<pinref part="OK1" gate="A" pin="A"/>
+<pinref part="GND" gate="A" pin="A"/>
 <wire x1="119.38" y1="43.18" x2="127" y2="43.18" width="0.1524" layer="91"/>
 </segment>
@@
 <segment>
 <wire x1="147.32" y1="48.26" x2="147.32" y2="43.18" width="0.1524" layer="91"/>
-<pinref part="OK1" gate="A" pin="COL"/>
+<pinref part="GND" gate="A" pin="COL"/>
 <wire x1="147.32" y1="43.18" x2="144.78" y2="43.18" width="0.1524" layer="91"/>
 <label x="147.32" y="48.26" size="1.778" layer="95"/>
@@
 <net name="SINAL_SKIB1" class="0">
 <segment>
-<pinref part="OK1" gate="A" pin="EMIT"/>
+<pinref part="GND" gate="A" pin="EMIT"/>
 <wire x1="144.78" y1="38.1" x2="147.32" y2="38.1" width="0.1524" layer="91"/>
 <wire x1="147.32" y1="38.1" x2="147.32" y2="30.48" width="0.1524" layer="91"/>
@@
 <pinref part="R7" gate="G$1" pin="2"/>
 <wire x1="101.6" y1="-15.24" x2="101.6" y2="-20.32" width="0.1524" layer="91"/>
-<pinref part="LED2" gate="G$1" pin="A"/>
+<pinref part="LSKIB2" gate="G$1" pin="A"/>
 <wire x1="101.6" y1="-20.32" x2="104.14" y2="-20.32" width="0.1524" layer="91"/>
 </segment>

Commit message: correções avionica e paraquedas
Parts:
- removed U$1, U$2: JST2.54X2P, CRD:JST2.54X2P
- added 3.3-BUZ, S1-S2, SK1-SK2: (no value), SparkFun-Connectors:CONN_022.54MM_SCREWTERM
- added OP1: PC817, optocoupler:PC817
- GND: value PC817 -> (none); device optocoupler:PC817 -> SparkFun-Connectors:CONN_022.54MM_SCREWTERM
- renumbered OK2 to OP2, SP2 to SP
Connections:
- net 3.3V: now also 3.3-BUZ.2, OP1.COL; no longer GND.COL, U$1.2
- net BUZZER: now also 3.3-BUZ.1, R4.2; no longer U$1.1
- net GND: now also GND.1, GND.2, OP1.C, R2.1, R3.1, R4.1; no longer GND.C
- net N$4: now also OP1.A; no longer GND.A
- net SINAL_SKIB1: now also OP1.EMIT, S1-S2.2; no longer GND.EMIT
- net SINAL_SKIB2: now also S1-S2.1
- net SKIB1: now also R2.2, SK1-SK2.2; no longer U$2.1
- net SKIB2: now also R3.2, SK1-SK2.1; no longer U$2.2
