File: Paraquedas/Paraquedas 2.1 - Corrosão A e B/Esquema.brd (EAGLE design)
At the start: 66 x 57.2 mm, 21 parts, among them Q1 IRF540, Q2 IRF540, Q3 IRF540

Commit message: Atualização de trilhas
Parts:
- added OP1: PC817, optocoupler:DIL04
- GND: value PC817 -> (none); device optocoupler:DIL04 -> SparkFun-Connectors:1X02_2.54_SCREWTERM
- moved GND 37.4 mm to (16.5, 7.62), turned to 0 degrees
- moved Q1 1.27 mm to (43.2, 26.7)
- moved R4 1.27 mm to (22.9, 12.7)
- flipped R2 to the top, turned to 0 degrees
- flipped R3 to the top, turned to 180 degrees
- renumbered J1 to S1-S2, J2 to SK1-SK2, J3 to 3.3-BUZ, OK2 to OP2, SP2 to SP
Connections:
- net 3.3V: now also OP1.4; no longer GND.4
- net GND: now also GND.P1, GND.P2, OP1.2; no longer GND.2
- net N$4: now also OP1.1; no longer GND.1
- net SINAL_SKIB1: now also OP1.3, S1-S2.P2; no longer GND.3, S1-S2.P1
- net SINAL_SKIB2: now also S1-S2.P1; no longer S1-S2.P2
- net SKIB1: now also SK1-SK2.P2; no longer SK1-SK2.P1
- net SKIB2: now also SK1-SK2.P1; no longer SK1-SK2.P2
Routing:
- net SINAL_SKIB2: track 15.3 -> 20.4 mm
- net SINAL_SKIB1: track 41.0 -> 44.8 mm
- net SKIB1: track 15.8 -> 17.6 mm
- net SKIB2: track 19.7 -> 20.2 mm
- net BUZZER: track 21.2 -> 20.7 mm
